File: hardware/boards/analog_i_rev4/analog/4-20mA.kicad_sch (KiCad schematic)
At the start: 9 parts, among them IC26001 INA826AIDR, IC32001 BD42540FJ-CE2, J26001 Screw_Terminal_01x03

Commit message: Analog I Rev 4.0.1 (#12)
## 2025-02-02 Hardware - Analog I Rev 4.0.1

### Changed - Hardware - Analog I Rev 4.0.1

* Replace input comparators with TLV3201s with 1M input pulldown to
resolve inadequate drive strength
    * Non-inverting hysteresis-free configuration
* Move screw terminal inward and place silkscreen terminal labels on the
outside
* Slightly widen board to make room for labels
* Update 3 pin screw terminal footprint for more accurate courtyard
* Update silkscreen labels to orient outward or toward the side opposite
the power/eth plugs
Parts:
- J26001: footprint TerminalBlock:TerminalBlock_bornier-3_P5.08mm -> aaa:Screw_Terminal_3_P5.08mm
Changed lines of the file:
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@@
 			)
 		)
-		(property "Footprint" "TerminalBlock:TerminalBlock_bornier-3_P5.08mm"
+		(property "Footprint" "aaa:Screw_Terminal_3_P5.08mm"
 			(at 76.2 102.87 0)
 			(effects
