File: hardware/boards/analog_i_rev5/analog/sk_1kHz.kicad_sch (KiCad schematic)
At the start: 6 parts, among them U9001 OPA333xxDBV

Commit message: update schematic with active filters and overvoltage protection
Parts:
- R9001, R9002: value 3.3k 1% -> 10k 1%; footprint Capacitor_SMD:C_0402_1005Metric -> Resistor_SMD:R_0402_1005Metric; LCSC C25890 -> C25744
Changed lines of the file:
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@@
 			)
 		)
-		(property "Value" "3.3k 1%"
+		(property "Value" "10k 1%"
 			(at 82.55 79.6544 90)
 			(effects
@@
 			)
 		)
-		(property "Footprint" "Capacitor_SMD:C_0402_1005Metric"
+		(property "Footprint" "Resistor_SMD:R_0402_1005Metric"
 			(at 82.55 82.55 0)
 			(effects
@@
 			)
 		)
-		(property "LCSC" "C25890"
+		(property "LCSC" "C25744"
 			(at 82.55 82.55 90)
 			(effects
@@
 			)
 		)
-		(property "Value" "3.3k 1%"
+		(property "Value" "10k 1%"
 			(at 93.98 79.6544 90)
 			(effects
@@
 			)
 		)
-		(property "Footprint" "Capacitor_SMD:C_0402_1005Metric"
+		(property "Footprint" "Resistor_SMD:R_0402_1005Metric"
 			(at 93.98 82.55 0)
 			(effects
@@
 			)
 		)
-		(property "LCSC" "C25890"
+		(property "LCSC" "C25744"
 			(at 93.98 82.55 90)
 			(effects

Commit message: limit amp voltage outputs to 3.3V
Connections:
- net +5V renamed +3V3
Changed lines of the file:
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@@
+	)
+	(symbol
+		(lib_id "power:+3V3")
+		(at 120.65 72.39 270)
+		(unit 1)
+		(exclude_from_sim no)
+		(in_bom yes)
+		(on_board yes)
+		(dnp no)
+		(property "Reference" "#PWR9003"
+			(at 116.84 72.39 0)
+			(effects
+				(font
+					(size 1.27 1.27)
+				)
+				(hide yes)
+			)
+		)
+		(property "Value" "+3V3"
+			(at 123.444 72.39 90)
+			(effects
+				(font
+					(size 1.27 1.27)
+				)
+				(justify left)
+			)
+		)
+		(property "Footprint" ""
+			(at 120.65 72.39 0)
+			(effects
+				(font
+					(size 1.27 1.27)
+				)
+				(hide yes)
+			)
+		)
+		(property "Datasheet" ""
+			(at 120.65 72.39 0)
+			(effects
+				(font
+					(size 1.27 1.27)
+				)
+				(hide yes)
+			)
+		)
+		(property "Description" "Power symbol creates a global label with name \"+3V3\""
+			(at 120.65 72.39 0)
+			(effects
+				(font
+					(size 1.27 1.27)
+				)
+				(hide yes)
+			)
+		)
+		(pin "1"
+		)
+		(instances
+			(project "analog_frontend_panel"
+				(path "/c241d083-1323-4b4a-a540-956d0afb7b72/10076f8f-acd4-4d92-be26-7bb7648716dd"
+					(reference "#PWR9003")
+					(unit 1)
+				)
+				(path "/c241d083-1323-4b4a-a540-956d0afb7b72/55b2a81f-7c95-46a9-b84c-c73547c2715f"
+					(reference "#PWR26003")
+					(unit 1)
+				)
+				(path "/c241d083-1323-4b4a-a540-956d0afb7b72/ecc8215c-aa73-4307-9e94-96da0574b4c2"
+					(reference "#PWR14003")
+					(unit 1)
+				)
+			)
+		)
 	)
 	(symbol
@@
 					(unit 1)
 				)
-			)
-		)
-	)
-	(symbol
-		(lib_id "power:+5V")
-		(at 120.65 72.39 270)
-		(unit 1)
-		(exclude_from_sim no)
-		(in_bom yes)
-		(on_board yes)
-		(dnp no)
-		(fields_autoplaced yes)
-		(property "Reference" "#PWR9003"
-			(at 116.84 72.39 0)
-			(effects
-				(font
-					(size 1.27 1.27)
-				)
-				(hide yes)
-			)
-		)
-		(property "Value" "+5V"
-			(at 123.952 72.3899 90)
-			(effects
-				(font
-					(size 1.27 1.27)
-				)
-				(justify left)
-			)
-		)
-		(property "Footprint" ""
-			(at 120.65 72.39 0)
-			(effects
-				(font
-					(size 1.27 1.27)
-				)
-				(hide yes)
-			)
-		)
-		(property "Datasheet" ""
-			(at 120.65 72.39 0)
-			(effects
-				(font
-					(size 1.27 1.27)
-				)
-				(hide yes)
-			)
-		)
-		(property "Description" "Power symbol creates a global label with name \"+5V\""
-			(at 120.65 72.39 0)
-			(effects
-				(font
-					(size 1.27 1.27)
-				)
-				(hide yes)
-			)
-		)
-		(pin "1"
-		)
-		(instances
-			(project "analog_frontend_panel"
-				(path "/c241d083-1323-4b4a-a540-956d0afb7b72/10076f8f-acd4-4d92-be26-7bb7648716dd"
-					(reference "#PWR9003")
-					(unit 1)
-				)
-				(path "/c241d083-1323-4b4a-a540-956d0afb7b72/55b2a81f-7c95-46a9-b84c-c73547c2715f"
-					(reference "#PWR27003")
-					(unit 1)
-				)
-				(path "/c241d083-1323-4b4a-a540-956d0afb7b72/ecc8215c-aa73-4307-9e94-96da0574b4c2"
-					(reference "#PWR14003")
-					(unit 1)
-				)
