File: hardware/boards/analog_i_rev5/analog/ain_g666p333_.kicad_sch (KiCad schematic)
At the start: 4 parts, among them IC32002 INA826AIDR

Commit message: remove redundant esd diodes
Changed lines of the file:
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@@
 	(wire
 		(pts
-			(xy 178.562 112.776) (xy 162.56 112.776)
+			(xy 162.56 112.776) (xy 162.56 103.124)
 		)
 		(stroke
@@
 	(wire
 		(pts
-			(xy 162.56 112.776) (xy 162.56 103.124)
+			(xy 162.56 112.776) (xy 178.562 112.776)
 		)
 		(stroke

Commit message: shorten board and update combined layout
Parts:
- renumbered C32005 to C36001, IC32002 to IC36001, R32003 to R36001, R32004 to R36002
Changed lines of the file:
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@@
 		(dnp no)
 		(fields_autoplaced yes)
-		(property "Reference" "#PWR32010"
+		(property "Reference" "#PWR209"
 			(at 158.496 114.554 0)
 			(effects
@@
 		)
 		(instances
+			(project "analog_i"
+				(path "/5a60c4b1-b6cb-416e-8883-8291fa089b87/c2baf18d-2b19-4edb-98b3-535275ee271f/ed60502d-2e6d-4293-85f2-5e967a3c42d8"
+					(reference "#PWR209")
+					(unit 1)
+				)
+			)
 			(project "analog_frontend_panel"
 				(path "/c241d083-1323-4b4a-a540-956d0afb7b72/ed60502d-2e6d-4293-85f2-5e967a3c42d8"
@@
 		(dnp no)
 		(fields_autoplaced yes)
-		(property "Reference" "IC32002"
+		(property "Reference" "IC36001"
 			(at 144.526 92.329 0)
 			(effects
@@
 		)
 		(instances
+			(project "analog_i"
+				(path "/5a60c4b1-b6cb-416e-8883-8291fa089b87/c2baf18d-2b19-4edb-98b3-535275ee271f/ed60502d-2e6d-4293-85f2-5e967a3c42d8"
+					(reference "IC36001")
+					(unit 1)
+				)
+			)
 			(project "analog_frontend_panel"
 				(path "/c241d083-1323-4b4a-a540-956d0afb7b72/ed60502d-2e6d-4293-85f2-5e967a3c42d8"
@@
 		(on_board yes)
 		(dnp no)
-		(property "Reference" "#PWR32012"
+		(property "Reference" "#PWR212"
 			(at 169.926 100.584 0)
 			(effects
@@
 		)
 		(instances
+			(project "analog_i"
+				(path "/5a60c4b1-b6cb-416e-8883-8291fa089b87/c2baf18d-2b19-4edb-98b3-535275ee271f/ed60502d-2e6d-4293-85f2-5e967a3c42d8"
+					(reference "#PWR212")
+					(unit 1)
+				)
+			)
 			(project "analog_frontend_panel"
 				(path "/c241d083-1323-4b4a-a540-956d0afb7b72/ed60502d-2e6d-4293-85f2-5e967a3c42d8"
@@
 		(on_board yes)
 		(dnp no)
-		(property "Reference" "R32003"
+		(property "Reference" "R36001"
 			(at 113.284 103.632 90)
 			(effects
@@
 		)
 		(instances
+			(project "analog_i"
+				(path "/5a60c4b1-b6cb-416e-8883-8291fa089b87/c2baf18d-2b19-4edb-98b3-535275ee271f/ed60502d-2e6d-4293-85f2-5e967a3c42d8"
+					(reference "R36001")
+					(unit 1)
+				)
+			)
 			(project "analog_frontend_panel"
 				(path "/c241d083-1323-4b4a-a540-956d0afb7b72/ed60502d-2e6d-4293-85f2-5e967a3c42d8"
@@
 		(on_board yes)
 		(dnp no)
-		(property "Reference" "R32004"
+		(property "Reference" "R36002"
 			(at 125.73 110.744 0)
 			(effects
@@
 		)
 		(instances
+			(project "analog_i"
+				(path "/5a60c4b1-b6cb-416e-8883-8291fa089b87/c2baf18d-2b19-4edb-98b3-535275ee271f/ed60502d-2e6d-4293-85f2-5e967a3c42d8"
+					(reference "R36002")
+					(unit 1)
+				)
+			)
 			(project "analog_frontend_panel"
 				(path "/c241d083-1323-4b4a-a540-956d0afb7b72/ed60502d-2e6d-4293-85f2-5e967a3c42d8"
@@
 		(on_board yes)
 		(dnp no)
-		(property "Reference" "#PWR32008"
+		(property "Reference" "#PWR210"
 			(at 124.46 119.634 0)
 			(effects
@@
 		)
 		(instances
+			(project "analog_i"
+				(path "/5a60c4b1-b6cb-416e-8883-8291fa089b87/c2baf18d-2b19-4edb-98b3-535275ee271f/ed60502d-2e6d-4293-85f2-5e967a3c42d8"
+					(reference "#PWR210")
+					(unit 1)
+				)
+			)
 			(project "analog_frontend_panel"
 				(path "/c241d083-1323-4b4a-a540-956d0afb7b72/ed60502d-2e6d-4293-85f2-5e967a3c42d8"
@@
 		(dnp no)
 		(fields_autoplaced yes)
-		(property "Reference" "#PWR32009"
+		(property "Reference" "#PWR211"
 			(at 124.206 100.584 0)
 			(effects
@@
 		)
 		(instances
+			(project "analog_i"
+				(path "/5a60c4b1-b6cb-416e-8883-8291fa089b87/c2baf18d-2b19-4edb-98b3-535275ee271f/ed60502d-2e6d-4293-85f2-5e967a3c42d8"
+					(reference "#PWR211")
+					(unit 1)
+				)
+			)
 			(project "analog_frontend_panel"
 				(path "/c241d083-1323-4b4a-a540-956d0afb7b72/ed60502d-2e6d-4293-85f2-5e967a3c42d8"
@@
 		(on_board yes)
 		(dnp no)
-		(property "Reference" "C32005"
+		(property "Reference" "C36001"
 			(at 168.656 96.266 90)
 			(effects
@@
 		)
 		(instances
+			(project "analog_i"
+				(path "/5a60c4b1-b6cb-416e-8883-8291fa089b87/c2baf18d-2b19-4edb-98b3-535275ee271f/ed60502d-2e6d-4293-85f2-5e967a3c42d8"
+					(reference "C36001")
+					(unit 1)
+				)
+			)
 			(project "analog_frontend_panel"
 				(path "/c241d083-1323-4b4a-a540-956d0afb7b72/ed60502d-2e6d-4293-85f2-5e967a3c42d8"
@@
 		(dnp no)
 		(fields_autoplaced yes)
-		(property "Reference" "#PWR32011"
+		(property "Reference" "#PWR213"
 			(at 168.656 112.014 0)
 			(effects
@@
 		)
 		(instances
-			(project "analog_frontend_panel"
-				(path "/c241d083-1323-4b4a-a540-956d0afb7b72/ed60502d-2e6d-4293-85f2-5e967a3c42d8"
+			(project "analog_i"
+				(path "/5a60c4b1-b6cb-416e-8883-8291fa089b87/c2baf18d-2b19-4edb-98b3-535275ee271f/ed60502d-2e6d-4293-85f2-5e967a3c42d8"
+					(reference "#PWR213")
+					(unit 1)
+				)
+			)
+			(project "analog_frontend_panel"
+				(path "/c241d083-1323-4b4a-a540-956d0afb7b72/ed60502d-2e6d-4293-85f2-5e967a3c42d8"
