File: hardware/boards/deimos_daq_rev5/analog/ktype_amp.kicad_sch (KiCad schematic)
At the start: 11 parts, among them IC9001 INA826AIDR, J9001 AM-K-PCB

Commit message: update changelog. rename hardware folder.
Changed lines of the file:
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@@
-	)
-	(symbol
-		(lib_id "power:GND")
-		(at 248.666 107.95 0)
-		(unit 1)
-		(exclude_from_sim no)
-		(in_bom yes)
-		(on_board yes)
-		(dnp no)
-		(property "Reference" "#PWR150"
-			(at 248.666 114.3 0)
-			(effects
-				(font
-					(size 1.27 1.27)
-				)
-				(hide yes)
-			)
-		)
-		(property "Value" "GND"
-			(at 250.444 112.014 0)
-			(effects
-				(font
-					(size 1.27 1.27)
-				)
-				(justify right)
-			)
-		)
-		(property "Footprint" ""
-			(at 248.666 107.95 0)
-			(effects
-				(font
-					(size 1.27 1.27)
-				)
-				(hide yes)
-			)
-		)
-		(property "Datasheet" ""
-			(at 248.666 107.95 0)
-			(effects
-				(font
-					(size 1.27 1.27)
-				)
-				(hide yes)
-			)
-		)
-		(property "Description" ""
-			(at 248.666 107.95 0)
-			(effects
-				(font
-					(size 1.27 1.27)
-				)
-				(hide yes)
-			)
-		)
-		(pin "1"
-		)
-		(instances
-			(project "analog_i"
-				(path "/5a60c4b1-b6cb-416e-8883-8291fa089b87/c2baf18d-2b19-4edb-98b3-535275ee271f/15b6c474-02be-417e-bc87-8489b7b45186"
-					(reference "#PWR150")
-					(unit 1)
-				)
-				(path "/5a60c4b1-b6cb-416e-8883-8291fa089b87/c2baf18d-2b19-4edb-98b3-535275ee271f/3688ccee-a1b0-41d3-bce5-95bc73998b83"
-					(reference "#PWR163")
-					(unit 1)
-				)
-			)
-			(project "analog_frontend_panel"
-				(path "/c241d083-1323-4b4a-a540-956d0afb7b72/15b6c474-02be-417e-bc87-8489b7b45186"
-					(reference "#PWR6002")
-					(unit 1)
-				)
-				(path "/c241d083-1323-4b4a-a540-956d0afb7b72/3688ccee-a1b0-41d3-bce5-95bc73998b83"
-					(reference "#PWR7002")
-					(unit 1)
-				)
-			)
-		)
 	)
 	(symbol

Commit message: put +/12V on all inamps. add 3.3V zener behind first resistor of each filter.
Parts:
- added C6001: 0.1uF, Capacitor_SMD:C_0402_1005Metric, symbol Device:C_Small
Connections:
- net GND: now also C6001.1; no longer IC9001.5 (-VS)
- net +3V3 renamed +12V
- new net -12V: C6001.2, IC9001.5 (-VS)
Changed lines of the file:
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@@
 	(paper "A4")
+	(junction
+		(at 220.472 105.41)
+		(diameter 0)
+		(color 0 0 0 0)
+	)
 	(junction
 		(at 124.46 104.14)
@@
 		(pts
 			(xy 219.71 102.87) (xy 232.664 102.87)
+		)
+		(stroke
+			(width 0)
+			(type default)
+		)
+	)
+	(wire
+		(pts
+			(xy 220.472 105.41) (xy 222.758 105.41)
+		)
+		(stroke
+			(width 0)
+			(type default)
+		)
+	)
+	(wire
+		(pts
+			(xy 219.71 105.41) (xy 220.472 105.41)
 		)
 		(stroke
@@
 	)
 	(symbol
+		(lib_id "power:GND")
+		(at 220.472 110.49 0)
+		(unit 1)
+		(exclude_from_sim no)
+		(in_bom yes)
+		(on_board yes)
+		(dnp no)
+		(property "Reference" "#PWR6003"
+			(at 220.472 116.84 0)
+			(effects
+				(font
+					(size 1.27 1.27)
+				)
+				(hide yes)
+			)
+		)
+		(property "Value" "GND"
+			(at 222.758 114.3 0)
+			(effects
+				(font
+					(size 1.27 1.27)
+				)
+				(justify right)
+			)
+		)
+		(property "Footprint" ""
+			(at 220.472 110.49 0)
+			(effects
+				(font
+					(size 1.27 1.27)
+				)
+				(hide yes)
+			)
+		)
+		(property "Datasheet" ""
+			(at 220.472 110.49 0)
+			(effects
+				(font
+					(size 1.27 1.27)
+				)
+				(hide yes)
+			)
+		)
+		(property "Description" ""
+			(at 220.472 110.49 0)
+			(effects
+				(font
+					(size 1.27 1.27)
+				)
+				(hide yes)
+			)
+		)
+		(pin "1"
+		)
+		(instances
+			(project "analog_frontend_panel"
+				(path "/c241d083-1323-4b4a-a540-956d0afb7b72/15b6c474-02be-417e-bc87-8489b7b45186"
+					(reference "#PWR6003")
+					(unit 1)
+				)
+				(path "/c241d083-1323-4b4a-a540-956d0afb7b72/3688ccee-a1b0-41d3-bce5-95bc73998b83"
+					(reference "#PWR7003")
+					(unit 1)
+				)
+			)
+		)
+	)
+	(symbol
 		(lib_id "Device:C_Small")
 		(at 232.664 105.41 180)
@@
 	)
 	(symbol
-		(lib_id "power:+3V3")
-		(at 228.6 97.79 270)
+		(lib_id "power:-12V")
+		(at 222.758 105.41 270)
 		(unit 1)
 		(exclude_from_sim no)
@@
 		(on_board yes)
 		(dnp no)
-		(property "Reference" "#PWR158"
-			(at 224.79 97.79 0)
-			(effects
-				(font
-					(size 1.27 1.27)
-				)
-				(hide yes)
-			)
-		)
-		(property "Value" "+3V3"
-			(at 231.394 97.79 90)
+		(property "Reference" "#PWR6001"
+			(at 218.948 105.41 0)
+			(effects
+				(font
+					(size 1.27 1.27)
+				)
+				(hide yes)
+			)
+		)
+		(property "Value" "-12V"
+			(at 221.234 107.442 90)
 			(effects
 				(font
@@
 		)
 		(property "Footprint" ""
-			(at 228.6 97.79 0)
+			(at 222.758 105.41 0)
 			(effects
 				(font
@@
 		)
 		(property "Datasheet" ""
-			(at 228.6 97.79 0)
-			(effects
-				(font
-					(size 1.27 1.27)
-				)
-				(hide yes)
-			)
-		)
-		(property "Description" "Power symbol creates a global label with name \"+3V3\""
-			(at 228.6 97.79 0)
+			(at 222.758 105.41 0)
+			(effects
+				(font
+					(size 1.27 1.27)
+				)
+				(hide yes)
+			)
+		)
+		(property "Description" "Power symbol creates a global label with name \"-12V\""
+			(at 222.758 105.41 0)
 			(effects
 				(font
@@
 		)
 		(instances
-			(project "analog_i"
-				(path "/5a60c4b1-b6cb-416e-8883-8291fa089b87/c2baf18d-2b19-4edb-98b3-535275ee271f/15b6c474-02be-417e-bc87-8489b7b45186"
-					(reference "#PWR158")
-					(unit 1)
-				)
-				(path "/5a60c4b1-b6cb-416e-8883-8291fa089b87/c2baf18d-2b19-4edb-98b3-535275ee271f/3688ccee-a1b0-41d3-bce5-95bc73998b83"
-					(reference "#PWR164")
-					(unit 1)
-				)
-			)
-			(project "analog_frontend_panel"
+			(project ""
 				(path "/c241d083-1323-4b4a-a540-956d0afb7b72/15b6c474-02be-417e-bc87-8489b7b45186"
 					(reference "#PWR6001")
@@
 	)
 	(symbol
+		(lib_id "power:+12V")
+		(at 228.6 97.79 270)
+		(unit 1)
+		(exclude_from_sim no)
+		(in_bom yes)
+		(on_board yes)
+		(dnp no)
+		(property "Reference" "#PWR6002"
+			(at 224.79 97.79 0)
+			(effects
+				(font
+					(size 1.27 1.27)
+				)
+				(hide yes)
+			)
+		)
+		(property "Value" "+12V"
+			(at 226.822 95.504 90)
+			(effects
+				(font
+					(size 1.27 1.27)
+				)
+				(justify left)
+			)
+		)
+		(property "Footprint" ""
+			(at 228.6 97.79 0)
+			(effects
+				(font
+					(size 1.27 1.27)
+				)
+				(hide yes)
+			)
+		)
+		(property "Datasheet" ""
+			(at 228.6 97.79 0)
+			(effects
+				(font
+					(size 1.27 1.27)
+				)
+				(hide yes)
+			)
+		)
+		(property "Description" "Power symbol creates a global label with name \"+12V\""
+			(at 228.6 97.79 0)
+			(effects
+				(font
+					(size 1.27 1.27)
+				)
+				(hide yes)
+			)
+		)
+		(pin "1"
+		)
+		(instances
+			(project ""
+				(path "/c241d083-1323-4b4a-a540-956d0afb7b72/15b6c474-02be-417e-bc87-8489b7b45186"
+					(reference "#PWR6002")
+					(unit 1)
+				)
+				(path "/c241d083-1323-4b4a-a540-956d0afb7b72/3688ccee-a1b0-41d3-bce5-95bc73998b83"
+					(reference "#PWR7002")
+					(unit 1)
+				)
+			)
+		)
+	)
+	(symbol
 		(lib_id "power:GND")
 		(at 222.25 90.17 180)
@@
 	)
 	(symbol
-		(lib_id "power:GND")
-		(at 219.71 105.41 90)
+		(lib_id "Device:C_Small")
+		(at 220.472 107.95 180)
 		(unit 1)
 		(exclude_from_sim no)
@@
 		(on_board yes)
 		(dnp no)
-		(property "Reference" "#PWR09004"
-			(at 226.06 105.41 0)
-			(effects
-				(font
-					(size 1.27 1.27)
-				)
-				(hide yes)
-			)
-		)
-		(property "Value" "GND"
-			(at 219.456 108.204 90)
-			(effects
-				(font
-					(size 1.27 1.27)
-				)
-				(justify right)
-			)
-		)
-		(property "Footprint" ""
-			(at 219.71 105.41 0)
-			(effects
-				(font
-					(size 1.27 1.27)
-				)
-				(hide yes)
-			)
-		)
-		(property "Datasheet" ""
-			(at 219.71 105.41 0)
+		(property "Reference" "C6001"
+			(at 215.138 110.998 90)
+			(effects
+				(font
+					(size 1.27 1.27)
+				)
+			)
+		)
+		(property "Value" "0.1uF"
+			(at 217.678 110.998 90)
+			(effects
+				(font
+					(size 1.27 1.27)
+				)
+			)
+		)
+		(property "Footprint" "Capacitor_SMD:C_0402_1005Metric"
+			(at 220.472 107.95 0)
+			(effects
+				(font
+					(size 1.27 1.27)
+				)
+				(hide yes)
+			)
+		)
+		(property "Datasheet" "~"
+			(at 220.472 107.95 0)
 			(effects
 				(font
@@
 		)
 		(property "Description" ""
-			(at 219.71 105.41 0)
+			(at 220.472 107.95 0)
 			(effects
 				(font
@@
 		(pin "1"
 		)
+		(pin "2"
+		)
 		(instances
-			(project "simplicity_analog_1"
-				(path "/5a60c4b1-b6cb-416e-8883-8291fa089b87/c2baf18d-2b19-4edb-98b3-535275ee271f/15b6c474-02be-417e-bc87-8489b7b45186"
-					(reference "#PWR09004")
-					(unit 1)
-				)
-				(path "/5a60c4b1-b6cb-416e-8883-8291fa089b87/c2baf18d-2b19-4edb-98b3-535275ee271f/3688ccee-a1b0-41d3-bce5-95bc73998b83"
-					(reference "#PWR015004")
-					(unit 1)
-				)
-			)
 			(project "analog_frontend_panel"
 				(path "/c241d083-1323-4b4a-a540-956d0afb7b72/15b6c474-02be-417e-bc87-8489b7b45186"
-					(reference "#PWR018")
+					(reference "C6001")
 					(unit 1)
 				)
 				(path "/c241d083-1323-4b4a-a540-956d0afb7b72/3688ccee-a1b0-41d3-bce5-95bc73998b83"
-					(reference "#PWR025")
-					(unit 1)
-				)
+					(reference "C7001")
+					(unit 1)
+				)

Commit message: add stabilizing integrator to current sinks
Other:
- moved on the sheet: C6001, C9004
Changed lines of the file:
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@@
 	(paper "A4")
-	(junction
-		(at 220.472 105.41)
-		(diameter 0)
-		(color 0 0 0 0)
-	)
 	(junction
 		(at 124.46 104.14)
@@
 	)
 	(junction
-		(at 222.25 97.79)
+		(at 219.71 97.79)
 		(diameter 0)
 		(color 0 0 0 0)
@@
 	)
 	(junction
+		(at 219.71 105.41)
+		(diameter 0)
+		(color 0 0 0 0)
+	)
+	(junction
 		(at 124.46 91.44)
 		(diameter 0)
@@
 	(wire
 		(pts
-			(xy 222.25 97.79) (xy 222.25 95.25)
+			(xy 113.03 104.14) (xy 116.84 104.14)
 		)
 		(stroke
@@
 	(wire
 		(pts
-			(xy 113.03 104.14) (xy 116.84 104.14)
+			(xy 219.71 100.33) (xy 252.73 100.33)
 		)
 		(stroke
@@
 	(wire
 		(pts
-			(xy 219.71 100.33) (xy 252.73 100.33)
+			(xy 124.46 95.25) (xy 124.46 91.44)
 		)
 		(stroke
@@
 	(wire
 		(pts
-			(xy 124.46 95.25) (xy 124.46 91.44)
+			(xy 113.03 91.44) (xy 124.46 91.44)
 		)
 		(stroke
@@
 	(wire
 		(pts
-			(xy 113.03 91.44) (xy 124.46 91.44)
+			(xy 175.26 100.33) (xy 175.26 102.87)
 		)
 		(stroke
@@
 	(wire
 		(pts
-			(xy 175.26 100.33) (xy 175.26 102.87)
+			(xy 189.23 96.52) (xy 192.024 96.52)
 		)
 		(stroke
@@
 	(wire
 		(pts
-			(xy 219.71 97.79) (xy 222.25 97.79)
+			(xy 116.84 104.14) (xy 124.46 104.14)
 		)
 		(stroke
@@
 	(wire
 		(pts
-			(xy 222.25 97.79) (xy 228.6 97.79)
+			(xy 180.34 100.33) (xy 191.77 100.33)
 		)
 		(stroke
@@
 	(wire
 		(pts
-			(xy 116.84 104.14) (xy 124.46 104.14)
-		)
-		(stroke
-			(width 0)
-			(type default)
-		)
-	)
-	(wire
-		(pts
-			(xy 180.34 100.33) (xy 191.77 100.33)
-		)
-		(stroke
-			(width 0)
-			(type default)
-		)
-	)
-	(wire
-		(pts
 			(xy 219.71 102.87) (xy 232.664 102.87)
-		)
-		(stroke
-			(width 0)
-			(type default)
-		)
-	)
-	(wire
-		(pts
-			(xy 220.472 105.41) (xy 222.758 105.41)
-		)
-		(stroke
-			(width 0)
-			(type default)
-		)
-	)
-	(wire
-		(pts
-			(xy 219.71 105.41) (xy 220.472 105.41)
 		)
 		(stroke
@@
 	(symbol
 		(lib_id "power:GND")
-		(at 220.472 110.49 0)
+		(at 219.71 110.49 0)
 		(unit 1)
 		(exclude_from_sim no)
@@
 		(dnp no)
 		(property "Reference" "#PWR6003"
-			(at 220.472 116.84 0)
+			(at 219.71 116.84 0)
 			(effects
 				(font
@@
 		)
 		(property "Value" "GND"
-			(at 222.758 114.3 0)
+			(at 221.996 114.3 0)
 			(effects
 				(font
@@
 		)
 		(property "Footprint" ""
-			(at 220.472 110.49 0)
+			(at 219.71 110.49 0)
 			(effects
 				(font
@@
 		)
 		(property "Datasheet" ""
-			(at 220.472 110.49 0)
+			(at 219.71 110.49 0)
 			(effects
 				(font
@@
 		)
 		(property "Description" ""
-			(at 220.472 110.49 0)
+			(at 219.71 110.49 0)
 			(effects
 				(font
@@
 		(on_board yes)
 		(dnp no)
-		(fields_autoplaced yes)
 		(property "Reference" "C9006"
-			(at 226.314 105.4037 90)
+			(at 235.966 105.918 90)
 			(effects
 				(font
@@
 		)
 		(property "Value" "0.1uF"
-			(at 228.854 105.4037 90)
+			(at 229.87 105.41 90)
 			(effects
 				(font
@@
 	(symbol
 		(lib_id "power:-12V")
-		(at 222.758 105.41 270)
+		(at 219.71 105.41 270)
 		(unit 1)
 		(exclude_from_sim no)
@@
 		(dnp no)
 		(property "Reference" "#PWR6001"
-			(at 218.948 105.41 0)
+			(at 215.9 105.41 0)
 			(effects
 				(font
@@
 		)
 		(property "Value" "-12V"
-			(at 221.234 107.442 90)
+			(at 222.504 105.41 90)
 			(effects
 				(font
@@
 		)
 		(property "Footprint" ""
-			(at 222.758 105.41 0)
+			(at 219.71 105.41 0)
 			(effects
 				(font
@@
 		)
 		(property "Datasheet" ""
-			(at 222.758 105.41 0)
+			(at 219.71 105.41 0)
 			(effects
 				(font
@@
 		)
 		(property "Description" "Power symbol creates a global label with name \"-12V\""
-			(at 222.758 105.41 0)
+			(at 219.71 105.41 0)
 			(effects
 				(font
@@
 	(symbol
 		(lib_id "Device:C_Small")
-		(at 222.25 92.71 180)
+		(at 219.71 95.25 180)
 		(unit 1)
 		(exclude_from_sim no)
@@
 		(dnp no)
 		(property "Reference" "C9004"
-			(at 217.17 91.44 0)
+			(at 222.25 96.012 90)
 			(effects
 				(font
@@
 		)
 		(property "Value" "0.1uF"
-			(at 214.63 93.98 0)
+			(at 216.916 96.012 90)
 			(effects
 				(font
@@
 		)
 		(property "Footprint" "Capacitor_SMD:C_0402_1005Metric"
-			(at 222.25 92.71 0)
+			(at 219.71 95.25 0)
 			(effects
 				(font
@@
 		)
 		(property "Datasheet" "~"
-			(at 222.25 92.71 0)
+			(at 219.71 95.25 0)
 			(effects
 				(font
@@
 		)
 		(property "Description" ""
-			(at 222.25 92.71 0)
+			(at 219.71 95.25 0)
 			(effects
 				(font
@@
 	(symbol
 		(lib_id "power:+12V")
-		(at 228.6 97.79 270)
+		(at 219.71 97.79 270)
 		(unit 1)
 		(exclude_from_sim no)
@@
 		(dnp no)
 		(property "Reference" "#PWR6002"
-			(at 224.79 97.79 0)
+			(at 215.9 97.79 0)
 			(effects
 				(font
@@
 		)
 		(property "Value" "+12V"
-			(at 226.822 95.504 90)
+			(at 222.504 97.536 90)
 			(effects
 				(font
@@
 		)
 		(property "Footprint" ""
-			(at 228.6 97.79 0)
+			(at 219.71 97.79 0)
 			(effects
 				(font
@@
 		)
 		(property "Datasheet" ""
-			(at 228.6 97.79 0)
+			(at 219.71 97.79 0)
 			(effects
 				(font
@@
 		)
 		(property "Description" "Power symbol creates a global label with name \"+12V\""
-			(at 228.6 97.79 0)
+			(at 219.71 97.79 0)
 			(effects
 				(font
@@
 	(symbol
 		(lib_id "power:GND")
-		(at 222.25 90.17 180)
+		(at 219.71 92.71 180)
 		(unit 1)
 		(exclude_from_sim no)
@@
 		(dnp no)
 		(property "Reference" "#PWR09005"
-			(at 222.25 83.82 0)
+			(at 219.71 86.36 0)
 			(effects
 				(font
@@
 		)
 		(property "Value" "GND"
-			(at 222.123 86.9188 90)
+			(at 219.583 89.4588 90)
 			(effects
 				(font
@@
 		)
 		(property "Footprint" ""
-			(at 222.25 90.17 0)
+			(at 219.71 92.71 0)
 			(effects
 				(font
@@
 		)
 		(property "Datasheet" ""
-			(at 222.25 90.17 0)
+			(at 219.71 92.71 0)
 			(effects
 				(font
@@
 		)
 		(property "Description" ""
-			(at 222.25 90.17 0)
+			(at 219.71 92.71 0)
 			(effects
 				(font
@@
 	(symbol
 		(lib_id "Device:C_Small")
-		(at 220.472 107.95 180)
+		(at 219.71 107.95 180)
 		(unit 1)
 		(exclude_from_sim no)
@@
 		(dnp no)
 		(property "Reference" "C6001"
-			(at 215.138 110.998 90)
+			(at 214.376 110.998 90)
 			(effects
 				(font
@@
 		)
 		(property "Value" "0.1uF"
-			(at 217.678 110.998 90)
+			(at 216.916 110.998 90)
 			(effects
 				(font
@@
 		)
 		(property "Footprint" "Capacitor_SMD:C_0402_1005Metric"
-			(at 220.472 107.95 0)
+			(at 219.71 107.95 0)
 			(effects
 				(font
@@
 		)
 		(property "Datasheet" "~"
-			(at 220.472 107.95 0)
+			(at 219.71 107.95 0)
 			(effects
 				(font
@@
 		)
 		(property "Description" ""
-			(at 220.472 107.95 0)
-			(effects
-				(font
+			(at 219.71 107.95 0)
+			(effects
+				(font

Commit message: use opa196 with split rail instead of opa333 with single rail. replace zeners.
Changed lines of the file:
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@@
-	(wire
-		(pts
-			(xy 189.23 96.52) (xy 192.024 96.52)
-		)
-		(stroke
-			(width 0)
-			(type default)
-		)
-	)
 	(wire
 		(pts

Commit message: restore rev5 and make this rev rev6
Parts:
- removed C6001: 0.1uF, Capacitor_SMD:C_0402_1005Metric, symbol Device:C_Small
Connections:
- net -12V is gone; now on net GND: IC9001.5 (-VS)
- net +12V renamed +3V3
Other:
- moved on the sheet: C9004
