File: hardware/boards/deimos_daq_rev6/analog/ain_g25p7_.kicad_sch (KiCad schematic)
At the start: 6 parts, among them IC38001 INA826AIDR

Commit message: exclude testpoints from BOM
Parts:
- renumbered C33007 to C38002, C33006 to C38003
Changed lines of the file:
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@@
 		(on_board yes)
 		(dnp no)
-		(property "Reference" "#PWR33012"
+		(property "Reference" "#PWR326"
 			(at 154.94 112.268 0)
 			(effects
@@
 		)
 		(instances
+			(project "analog_i"
+				(path "/5a60c4b1-b6cb-416e-8883-8291fa089b87/c2baf18d-2b19-4edb-98b3-535275ee271f/a1ee2b3a-0c82-480a-bd10-9f01e8ac3dcc"
+					(reference "#PWR326")
+					(unit 1)
+				)
+			)
 			(project ""
 				(path "/c241d083-1323-4b4a-a540-956d0afb7b72/a1ee2b3a-0c82-480a-bd10-9f01e8ac3dcc"
@@
 		(on_board yes)
 		(dnp no)
-		(property "Reference" "#PWR33013"
+		(property "Reference" "#PWR324"
 			(at 154.94 104.648 0)
 			(effects
@@
 		)
 		(instances
+			(project "analog_i"
+				(path "/5a60c4b1-b6cb-416e-8883-8291fa089b87/c2baf18d-2b19-4edb-98b3-535275ee271f/a1ee2b3a-0c82-480a-bd10-9f01e8ac3dcc"
+					(reference "#PWR324")
+					(unit 1)
+				)
+			)
 			(project ""
 				(path "/c241d083-1323-4b4a-a540-956d0afb7b72/a1ee2b3a-0c82-480a-bd10-9f01e8ac3dcc"
@@
 		(on_board yes)
 		(dnp no)
-		(property "Reference" "C33006"
+		(property "Reference" "C38003"
 			(at 170.434 115.062 90)
 			(effects
@@
 		)
 		(instances
+			(project "analog_i"
+				(path "/5a60c4b1-b6cb-416e-8883-8291fa089b87/c2baf18d-2b19-4edb-98b3-535275ee271f/a1ee2b3a-0c82-480a-bd10-9f01e8ac3dcc"
+					(reference "C38003")
+					(unit 1)
+				)
+			)
 			(project "analog_frontend_panel"
 				(path "/c241d083-1323-4b4a-a540-956d0afb7b72/a1ee2b3a-0c82-480a-bd10-9f01e8ac3dcc"
@@
 		(on_board yes)
 		(dnp no)
-		(property "Reference" "C33007"
+		(property "Reference" "C38002"
 			(at 161.29 116.586 90)
 			(effects
@@
 		)
 		(instances
+			(project "analog_i"
+				(path "/5a60c4b1-b6cb-416e-8883-8291fa089b87/c2baf18d-2b19-4edb-98b3-535275ee271f/a1ee2b3a-0c82-480a-bd10-9f01e8ac3dcc"
+					(reference "C38002")
+					(unit 1)
+				)
+			)
 			(project "analog_frontend_panel"
 				(path "/c241d083-1323-4b4a-a540-956d0afb7b72/a1ee2b3a-0c82-480a-bd10-9f01e8ac3dcc"
@@
 		(dnp no)
 		(fields_autoplaced yes)
-		(property "Reference" "#PWR33011"
+		(property "Reference" "#PWR325"
 			(at 158.75 123.698 0)
 			(effects
@@
 		)
 		(instances
+			(project "analog_i"
+				(path "/5a60c4b1-b6cb-416e-8883-8291fa089b87/c2baf18d-2b19-4edb-98b3-535275ee271f/a1ee2b3a-0c82-480a-bd10-9f01e8ac3dcc"
+					(reference "#PWR325")
+					(unit 1)
+				)
+			)
 			(project "analog_frontend_panel"
 				(path "/c241d083-1323-4b4a-a540-956d0afb7b72/a1ee2b3a-0c82-480a-bd10-9f01e8ac3dcc"
@@
 		(on_board yes)
 		(dnp no)
-		(property "Reference" "#PWR33010"
+		(property "Reference" "#PWR327"
 			(at 167.64 121.158 0)
 			(effects
@@
 		)
 		(instances
+			(project "analog_i"
+				(path "/5a60c4b1-b6cb-416e-8883-8291fa089b87/c2baf18d-2b19-4edb-98b3-535275ee271f/a1ee2b3a-0c82-480a-bd10-9f01e8ac3dcc"
+					(reference "#PWR327")
+					(unit 1)
+				)
+			)
 			(project "analog_frontend_panel"
 				(path "/c241d083-1323-4b4a-a540-956d0afb7b72/a1ee2b3a-0c82-480a-bd10-9f01e8ac3dcc"
