File: hardware/boards/deimos_daq_rev6/analog/dac_buf.kicad_sch (KiCad schematic)
At the start: 4 parts, among them IC53001 INA826AIDR

Commit message: exclude testpoints from BOM
Parts:
- renumbered C39003 to C53002
Changed lines of the file:
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@@
 		(on_board yes)
 		(dnp no)
-		(property "Reference" "C39003"
+		(property "Reference" "C53002"
 			(at 158.242 111.506 90)
 			(effects
@@
 		)
 		(instances
+			(project "analog_i"
+				(path "/5a60c4b1-b6cb-416e-8883-8291fa089b87/c2baf18d-2b19-4edb-98b3-535275ee271f/13efaa5b-e400-45cc-91a0-978d4e7725f3"
+					(reference "C53002")
+					(unit 1)
+				)
+				(path "/5a60c4b1-b6cb-416e-8883-8291fa089b87/c2baf18d-2b19-4edb-98b3-535275ee271f/cebae258-d5b5-4a87-b6e3-430d71499c69"
+					(reference "C54002")
+					(unit 1)
+				)
+			)
 			(project "analog_frontend_panel"
 				(path "/c241d083-1323-4b4a-a540-956d0afb7b72/13efaa5b-e400-45cc-91a0-978d4e7725f3"
@@
 		(dnp no)
 		(fields_autoplaced yes)
-		(property "Reference" "#PWR39011"
+		(property "Reference" "#PWR358"
 			(at 151.384 98.298 0)
 			(effects
@@
 		)
 		(instances
+			(project "analog_i"
+				(path "/5a60c4b1-b6cb-416e-8883-8291fa089b87/c2baf18d-2b19-4edb-98b3-535275ee271f/13efaa5b-e400-45cc-91a0-978d4e7725f3"
+					(reference "#PWR358")
+					(unit 1)
+				)
+				(path "/5a60c4b1-b6cb-416e-8883-8291fa089b87/c2baf18d-2b19-4edb-98b3-535275ee271f/cebae258-d5b5-4a87-b6e3-430d71499c69"
+					(reference "#PWR361")
+					(unit 1)
+				)
+			)
 			(project ""
 				(path "/c241d083-1323-4b4a-a540-956d0afb7b72/13efaa5b-e400-45cc-91a0-978d4e7725f3"
@@
 		(dnp no)
 		(fields_autoplaced yes)
-		(property "Reference" "#PWR39013"
+		(property "Reference" "#PWR359"
 			(at 155.194 117.348 0)
 			(effects
@@
 		)
 		(instances
+			(project "analog_i"
+				(path "/5a60c4b1-b6cb-416e-8883-8291fa089b87/c2baf18d-2b19-4edb-98b3-535275ee271f/13efaa5b-e400-45cc-91a0-978d4e7725f3"
+					(reference "#PWR359")
+					(unit 1)
+				)
+				(path "/5a60c4b1-b6cb-416e-8883-8291fa089b87/c2baf18d-2b19-4edb-98b3-535275ee271f/cebae258-d5b5-4a87-b6e3-430d71499c69"
+					(reference "#PWR362")
+					(unit 1)
+				)
+			)
 			(project "analog_frontend_panel"
 				(path "/c241d083-1323-4b4a-a540-956d0afb7b72/13efaa5b-e400-45cc-91a0-978d4e7725f3"
@@
 		(dnp no)
 		(fields_autoplaced yes)
-		(property "Reference" "#PWR39012"
+		(property "Reference" "#PWR360"
 			(at 151.384 105.918 0)
 			(effects
@@
 		)
 		(instances
+			(project "analog_i"
+				(path "/5a60c4b1-b6cb-416e-8883-8291fa089b87/c2baf18d-2b19-4edb-98b3-535275ee271f/13efaa5b-e400-45cc-91a0-978d4e7725f3"
+					(reference "#PWR360")
+					(unit 1)
+				)
+				(path "/5a60c4b1-b6cb-416e-8883-8291fa089b87/c2baf18d-2b19-4edb-98b3-535275ee271f/cebae258-d5b5-4a87-b6e3-430d71499c69"
+					(reference "#PWR363")
+					(unit 1)
+				)
+			)
 			(project ""
 				(path "/c241d083-1323-4b4a-a540-956d0afb7b72/13efaa5b-e400-45cc-91a0-978d4e7725f3"
