File: hardware/boards/deimos_daq_rev6/base/ethernet.kicad_sch (KiCad schematic)
At the start: 44 parts, among them J3001 RCH_RC01133, T1 H1102NLT, U5 LAN8742A, Y2 NX2016SA-25.000M-STD-CZS-1

Commit message: clean up ethernet layout. remove unnecessary phy crystal load caps.
Parts:
- removed C20, C21: 5.6pF 0402, Capacitor_SMD:C_0402_1005Metric, symbol Device:C_Small
