File: hardware/boards/deimos_daq_rev6/base/1v024_ref.kicad_sch (KiCad schematic)
At the start: 5 parts, among them IC5004 REF35102QDBVR

Commit message: Deimos DAQ Rev 6.0.1 (#30)
## 2025-10-12 deimos 0.11.2, deimos_shared 0.5.1, Deimos DAQ Rev 6.0.1
hardware and firmware

Tooling
* ubuntu 24.04
* kicad 8 with hierarchical PCB plugin
* protocase designer v7.2.1 linux version
* Run like
`LD_LIBRARY_PATH=/opt/protocasedesigner/lib/app/natives/occjava/linux-x86_64/
/opt/protocasedesigner/bin/ProtocaseDesigner` to resolve link path issue
for java runtime
* freecad 1.0.2

### Added

Hardware
* Deimos DAQ Rev 6.0.1 schematic and layout
* [x] Replace overvoltage protection diodes from leaky zeners to
low-leakage JFET clamp
* [x] Add 5V LDO as supply for resistance amplifiers to restore gate
voltage margin
* [x] Use smaller resistor values for resistance amp common-mode filter
* INA826 has significant input bias current (~25nA) which makes a
nontrivial voltage across 20k resistance
* [x] Disable internal buffer for DAC to allow rail-to-rail operation
        * Buffered mode min and max voltages are 20mV off the rails
* Can rely on external buffer that is already implemented for
overvoltage protection
* Controller Base Rev 16.0.1
    * [x] Remove unnecessary clamping diodes
    * [x] Remove unnecessary eth PHY crystal load caps
    * [x] Clean up ethernet layout

Software & Firmware
* deimos_daq_rev6 firmware
* Rolled forward to latest `interpn` and `flaw` versions w/ perf
improvements; ~30% increase in cycle timing margin
* deimos
    * Add rev 6 firmware and calc plugin
* deimos_shared
    * Add rev 6 packet formats

Analysis
* Added JFET diode clamp spice model
Parts:
- removed D7001: BZT52C3V3, Diode_SMD:D_SOD-323, symbol Device:D_Zener
Changed lines of the file:
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@@
 	(paper "A4")
-	(junction
-		(at 167.132 96.266)
-		(diameter 0)
-		(color 0 0 0 0)
-	)
-	(junction
-		(at 167.132 88.646)
-		(diameter 0)
-		(color 0 0 0 0)
-	)
 	(junction
 		(at 153.289 105.156)
@@
 	(wire
 		(pts
-			(xy 164.084 88.646) (xy 167.132 88.646)
-		)
-		(stroke
-			(width 0)
-			(type default)
-		)
-	)
-	(wire
-		(pts
-			(xy 164.084 96.266) (xy 167.132 96.266)
-		)
-		(stroke
-			(width 0)
-			(type default)
-		)
-	)
-	(wire
-		(pts
-			(xy 167.132 88.646) (xy 169.926 88.646)
-		)
-		(stroke
-			(width 0)
-			(type default)
-		)
-	)
-	(wire
-		(pts
-			(xy 164.084 93.726) (xy 164.084 96.266)
+			(xy 164.084 88.646) (xy 169.926 88.646)
 		)
 		(stroke
@@
 	(symbol
 		(lib_id "power:GND")
-		(at 167.132 96.266 0)
+		(at 164.084 93.726 0)
 		(unit 1)
 		(exclude_from_sim no)
@@
 		(dnp no)
 		(property "Reference" "#PWR05018"
-			(at 167.132 102.616 0)
+			(at 164.084 100.076 0)
 			(effects
 				(font
@@
 		)
 		(property "Value" "GND"
-			(at 167.132 103.886 90)
+			(at 162.052 97.282 0)
 			(effects
 				(font
@@
 		)
 		(property "Footprint" ""
-			(at 167.132 96.266 0)
+			(at 164.084 93.726 0)
 			(effects
 				(font
@@
 		)
 		(property "Datasheet" ""
-			(at 167.132 96.266 0)
+			(at 164.084 93.726 0)
 			(effects
 				(font
@@
 		)
 		(property "Description" ""
-			(at 167.132 96.266 0)
+			(at 164.084 93.726 0)
 			(effects
 				(font
@@
 					(unit 1)
 				)
-			)
-		)
-	)
-	(symbol
-		(lib_id "Device:D_Zener")
-		(at 167.132 92.456 270)
-		(unit 1)
-		(exclude_from_sim no)
-		(in_bom yes)
-		(on_board yes)
-		(dnp no)
-		(property "Reference" "D7001"
-			(at 164.338 92.456 0)
-			(effects
-				(font
-					(size 1.27 1.27)
-				)
-				(hide yes)
-			)
-		)
-		(property "Value" "BZT52C3V3"
-			(at 170.688 95.25 0)
-			(effects
-				(font
-					(size 1.27 1.27)
-				)
-			)
-		)
-		(property "Footprint" "Diode_SMD:D_SOD-323"
-			(at 167.132 92.456 0)
-			(effects
-				(font
-					(size 1.27 1.27)
-				)
-				(hide yes)
-			)
-		)
-		(property "Datasheet" "~"
-			(at 167.132 92.456 0)
-			(effects
-				(font
-					(size 1.27 1.27)
-				)
-				(hide yes)
-			)
-		)
-		(property "Description" ""
-			(at 167.132 92.456 0)
-			(effects
-				(font
-					(size 1.27 1.27)
-				)
-				(hide yes)
-			)
-		)
-		(property "LCSC" "C2112"
-			(at 167.132 92.456 0)
-			(effects
-				(font
-					(size 1.27 1.27)
-				)
-				(hide yes)
-			)
-		)
-		(pin "1"
-		)
-		(pin "2"
-		)
-		(instances
-			(project "stm32h7_base"
-				(path "/511605a4-f92c-43a6-a2c6-3cb535ac8a8e/a65c6055-0639-4361-905b-5a6b6f014124"
-					(reference "D7001")
-					(unit 1)
-				)
-			)
-			(project "analog_i"
-				(path "/5a60c4b1-b6cb-416e-8883-8291fa089b87/b545dc42-87cf-45f6-8889-98202e5f492a/a65c6055-0639-4361-905b-5a6b6f014124"
-					(reference "D5002")
-					(unit 1)
-				)
