File: hardware/boards/deimos_daq_rev7/analog/sk_3kHz.kicad_sch (KiCad schematic)
At the start: 9 parts, among them Q21001 MMBFJ113, Q21002 MMBFJ113, U21001 OPA196xDBV

Commit message: replace user power with gpio. wip to update frontend layout.
Parts:
- renumbered C27001 to C33001, C27002 to C33002, C21003 to C33003, C21004 to C33004, Q21001 to Q33001, Q21002 to Q33002, R27001 to R33001, R27002 to R33002, U21001 to U33001
Changed lines of the file:
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@@
 		(on_board yes)
 		(dnp no)
-		(property "Reference" "#PWR220"
+		(property "Reference" "#PWR286"
 			(at 113.03 88.9 0)
 			(effects
@@
 		(on_board yes)
 		(dnp no)
-		(property "Reference" "C27001"
+		(property "Reference" "C33001"
 			(at 106.68 96.012 90)
 			(effects
@@
 		(on_board yes)
 		(dnp no)
-		(property "Reference" "#PWR216"
+		(property "Reference" "#PWR283"
 			(at 92.964 110.49 0)
 			(effects
@@
 		(on_board yes)
 		(dnp no)
-		(property "Reference" "R27001"
+		(property "Reference" "R33001"
 			(at 82.55 77.343 90)
 			(effects
@@
 		(on_board yes)
 		(dnp no)
-		(property "Reference" "#PWR208"
+		(property "Reference" "#PWR278"
 			(at 124.46 92.71 0)
 			(effects
@@
 		(on_board yes)
 		(dnp no)
-		(property "Reference" "Q21001"
+		(property "Reference" "Q33001"
 			(at 80.772 100.584 90)
 			(effects
@@
 		(on_board yes)
 		(dnp no)
-		(property "Reference" "#PWR217"
+		(property "Reference" "#PWR285"
 			(at 80.518 100.584 0)
 			(effects
@@
 		(on_board yes)
 		(dnp no)
-		(property "Reference" "#PWR209"
+		(property "Reference" "#PWR280"
 			(at 124.46 77.47 0)
 			(effects
@@
 		(on_board yes)
 		(dnp no)
-		(property "Reference" "Q21002"
+		(property "Reference" "Q33002"
 			(at 92.964 91.44 90)
 			(effects
@@
 		(on_board yes)
 		(dnp no)
-		(property "Reference" "U21001"
+		(property "Reference" "U33001"
 			(at 107.442 78.994 0)
 			(effects
@@
 		(on_board yes)
 		(dnp no)
-		(property "Reference" "R27002"
+		(property "Reference" "R33002"
 			(at 93.98 77.343 90)
 			(effects
@@
 		(on_board yes)
 		(dnp no)
-		(property "Reference" "C21003"
+		(property "Reference" "C33003"
 			(at 119.38 81.788 90)
 			(effects
@@
 		(on_board yes)
 		(dnp no)
-		(property "Reference" "C21004"
+		(property "Reference" "C33004"
 			(at 118.872 97.536 90)
 			(effects
@@
 		(on_board yes)
 		(dnp no)
-		(property "Reference" "C27002"
+		(property "Reference" "C33002"
 			(at 111.252 65.532 90)
 			(effects
@@
 		(on_board yes)
 		(dnp no)
-		(property "Reference" "#PWR212"
+		(property "Reference" "#PWR281"
 			(at 113.03 81.28 0)
 			(effects
@@
 		(on_board yes)
 		(dnp no)
-		(property "Reference" "#PWR185"
+		(property "Reference" "#PWR200"
 			(at 101.6 99.06 0)
 			(effects

Commit message: flip pin order in symbol for pluggable terminal block
Parts:
- renumbered C33001 to C27001, C33002 to C27002, C33003 to C27003, C33004 to C27004, Q33001 to Q27001, Q33002 to Q27002, R33001 to R27001, R33002 to R27002, U33001 to U27001
Changed lines of the file:
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@@
 		(on_board yes)
 		(dnp no)
-		(property "Reference" "#PWR286"
+		(property "Reference" "#PWR246"
 			(at 113.03 88.9 0)
 			(effects
@@
 		(on_board yes)
 		(dnp no)
-		(property "Reference" "C33001"
+		(property "Reference" "C27001"
 			(at 106.68 96.012 90)
 			(effects
@@
 		(on_board yes)
 		(dnp no)
-		(property "Reference" "#PWR283"
+		(property "Reference" "#PWR244"
 			(at 92.964 110.49 0)
 			(effects
@@
 		(on_board yes)
 		(dnp no)
-		(property "Reference" "R33001"
+		(property "Reference" "R27001"
 			(at 82.55 77.343 90)
 			(effects
@@
 		(on_board yes)
 		(dnp no)
-		(property "Reference" "#PWR278"
+		(property "Reference" "#PWR239"
 			(at 124.46 92.71 0)
 			(effects
@@
 		(on_board yes)
 		(dnp no)
-		(property "Reference" "Q33001"
+		(property "Reference" "Q27001"
 			(at 80.772 100.584 90)
 			(effects
@@
 		(on_board yes)
 		(dnp no)
-		(property "Reference" "#PWR285"
+		(property "Reference" "#PWR245"
 			(at 80.518 100.584 0)
 			(effects
@@
 		(on_board yes)
 		(dnp no)
-		(property "Reference" "#PWR280"
+		(property "Reference" "#PWR242"
 			(at 124.46 77.47 0)
 			(effects
@@
 		(on_board yes)
 		(dnp no)
-		(property "Reference" "Q33002"
+		(property "Reference" "Q27002"
 			(at 92.964 91.44 90)
 			(effects
@@
 		(on_board yes)
 		(dnp no)
-		(property "Reference" "U33001"
+		(property "Reference" "U27001"
 			(at 107.442 78.994 0)
 			(effects
@@
 		(on_board yes)
 		(dnp no)
-		(property "Reference" "R33002"
+		(property "Reference" "R27002"
 			(at 93.98 77.343 90)
 			(effects
@@
 		(on_board yes)
 		(dnp no)
-		(property "Reference" "C33003"
+		(property "Reference" "C27003"
 			(at 119.38 81.788 90)
 			(effects
@@
 		(on_board yes)
 		(dnp no)
-		(property "Reference" "C33004"
+		(property "Reference" "C27004"
 			(at 118.872 97.536 90)
 			(effects
@@
 		(on_board yes)
 		(dnp no)
-		(property "Reference" "C33002"
+		(property "Reference" "C27002"
 			(at 111.252 65.532 90)
 			(effects
@@
 		(on_board yes)
 		(dnp no)
-		(property "Reference" "#PWR281"
+		(property "Reference" "#PWR243"
 			(at 113.03 81.28 0)
 			(effects
@@
 		(on_board yes)
 		(dnp no)
-		(property "Reference" "#PWR200"
+		(property "Reference" "#PWR185"
 			(at 101.6 99.06 0)
 			(effects

Commit message: update schematic with regulated OVP rail
Parts:
- renumbered C27001 to C35001, C27002 to C35002, C27003 to C35003, C27004 to C35004, Q27001 to Q35001, Q27002 to Q35002, R27002 to R35002, R27001 to R43001, U27001 to U35001
Connections:
- net +3V3 renamed 2V5_OVP
Changed lines of the file:
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@@
+	)
+	(junction
+		(at 93.218 89.916)
+		(diameter 0)
+		(color 0 0 0 0)
 	)
 	(junction
@@
 	)
 	(junction
-		(at 93.218 89.916)
-		(diameter 0)
-		(color 0 0 0 0)
-	)
-	(junction
 		(at 133.35 85.09)
 		(diameter 0)
@@
 	(wire
 		(pts
+			(xy 80.518 106.68) (xy 80.518 104.394)
+		)
+		(stroke
+			(width 0)
+			(type default)
+		)
+	)
+	(wire
+		(pts
 			(xy 75.438 97.79) (xy 75.438 104.394)
 		)
@@
 		(pts
 			(xy 133.35 99.06) (xy 133.35 85.09)
+		)
+		(stroke
+			(width 0)
+			(type default)
+		)
+	)
+	(wire
+		(pts
+			(xy 77.47 106.68) (xy 80.518 106.68)
 		)
 		(stroke
@@
 			)
 			(justify left)
+		)
+	)
+	(global_label "2V5_OVP"
+		(shape input)
+		(at 77.47 106.68 180)
+		(fields_autoplaced yes)
+		(effects
+			(font
+				(size 1.27 1.27)
+			)
+			(justify right)
+		)
+		(property "Intersheetrefs" "${INTERSHEET_REFS}"
+			(at 66.3205 106.68 0)
+			(effects
+				(font
+					(size 1.27 1.27)
+				)
+				(justify right)
+				(hide yes)
+			)
 		)
 	)
@@
 		(on_board yes)
 		(dnp no)
-		(property "Reference" "#PWR246"
+		(property "Reference" "#PWR309"
 			(at 113.03 88.9 0)
 			(effects
@@
 		(on_board yes)
 		(dnp no)
-		(property "Reference" "C27001"
+		(property "Reference" "C35001"
 			(at 106.68 96.012 90)
 			(effects
@@
 		(on_board yes)
 		(dnp no)
-		(property "Reference" "#PWR244"
+		(property "Reference" "#PWR305"
 			(at 92.964 110.49 0)
 			(effects
@@
 		(on_board yes)
 		(dnp no)
-		(property "Reference" "R27001"
+		(property "Reference" "R43001"
 			(at 82.55 77.343 90)
 			(effects
@@
 		(on_board yes)
 		(dnp no)
-		(property "Reference" "#PWR239"
+		(property "Reference" "#PWR300"
 			(at 124.46 92.71 0)
 			(effects
@@
 		(on_board yes)
 		(dnp no)
-		(property "Reference" "Q27001"
+		(property "Reference" "Q35001"
 			(at 80.772 100.584 90)
 			(effects
@@
 				(path "/c241d083-1323-4b4a-a540-956d0afb7b72/fb5bb440-61c9-4bd3-9ab6-a463ad90c8bb/413450a6-23f7-43dd-83b0-93f1b2a57e6d"
 					(reference "Q15001")
-					(unit 1)
-				)
-			)
-		)
-	)
-	(symbol
-		(lib_id "power:+3V3")
-		(at 80.518 104.394 180)
-		(unit 1)
-		(exclude_from_sim no)
-		(in_bom yes)
-		(on_board yes)
-		(dnp no)
-		(property "Reference" "#PWR245"
-			(at 80.518 100.584 0)
-			(effects
-				(font
-					(size 1.27 1.27)
-				)
-				(hide yes)
-			)
-		)
-		(property "Value" "+3V3"
-			(at 79.756 108.204 0)
-			(effects
-				(font
-					(size 1.27 1.27)
-				)
-			)
-		)
-		(property "Footprint" ""
-			(at 80.518 104.394 0)
-			(effects
-				(font
-					(size 1.27 1.27)
-				)
-				(hide yes)
-			)
-		)
-		(property "Datasheet" ""
-			(at 80.518 104.394 0)
-			(effects
-				(font
-					(size 1.27 1.27)
-				)
-				(hide yes)
-			)
-		)
-		(property "Description" "Power symbol creates a global label with name \"+3V3\""
-			(at 80.518 104.394 0)
-			(effects
-				(font
-					(size 1.27 1.27)
-				)
-				(hide yes)
-			)
-		)
-		(pin "1"
-		)
-		(instances
-			(project "analog_i"
-				(path "/5a60c4b1-b6cb-416e-8883-8291fa089b87/c2baf18d-2b19-4edb-98b3-535275ee271f/19141585-7846-417a-91df-f61215fe3233/413450a6-23f7-43dd-83b0-93f1b2a57e6d"
-					(reference "#PWR233")
-					(unit 1)
-				)
-				(path "/5a60c4b1-b6cb-416e-8883-8291fa089b87/c2baf18d-2b19-4edb-98b3-535275ee271f/1fbd3e63-3701-4f31-b722-16e65c25cea8/413450a6-23f7-43dd-83b0-93f1b2a57e6d"
-					(reference "#PWR245")
-					(unit 1)
-				)
-				(path "/5a60c4b1-b6cb-416e-8883-8291fa089b87/c2baf18d-2b19-4edb-98b3-535275ee271f/3b63f70a-358c-4846-8cdc-f459df41a6c2/0ab125f9-c5b5-4162-87a8-3c0a237e613b"
-					(reference "#PWR350")
-					(unit 1)
-				)
-				(path "/5a60c4b1-b6cb-416e-8883-8291fa089b87/c2baf18d-2b19-4edb-98b3-535275ee271f/77831b95-4af9-4be7-883d-350d130a19a2/4b0b4e20-0ae3-4a37-acd3-d6dca880b023"
-					(reference "#PWR270")
-					(unit 1)
-				)
-				(path "/5a60c4b1-b6cb-416e-8883-8291fa089b87/c2baf18d-2b19-4edb-98b3-535275ee271f/b7e73f80-a01f-409c-a1ae-634c4b865833/4b0b4e20-0ae3-4a37-acd3-d6dca880b023"
-					(reference "#PWR285")
-					(unit 1)
-				)
-				(path "/5a60c4b1-b6cb-416e-8883-8291fa089b87/c2baf18d-2b19-4edb-98b3-535275ee271f/be220027-a1e7-4f8a-b4af-8d208623fd51/dd604314-47f9-4977-b551-e4daf9b9f74b"
-					(reference "#PWR338")
-					(unit 1)
-				)
-				(path "/5a60c4b1-b6cb-416e-8883-8291fa089b87/c2baf18d-2b19-4edb-98b3-535275ee271f/c0b9347d-9aa2-441c-987f-68119b1d92c1/0ab125f9-c5b5-4162-87a8-3c0a237e613b"
-					(reference "#PWR356")
-					(unit 1)
-				)
-				(path "/5a60c4b1-b6cb-416e-8883-8291fa089b87/c2baf18d-2b19-4edb-98b3-535275ee271f/c99c1b0b-6659-4cec-a152-edd7ebc08576/4b0b4e20-0ae3-4a37-acd3-d6dca880b023"
-					(reference "#PWR306")
-					(unit 1)
-				)
-				(path "/5a60c4b1-b6cb-416e-8883-8291fa089b87/c2baf18d-2b19-4edb-98b3-535275ee271f/ed2f7b43-1244-451f-9def-7c9639b384e1/dd604314-47f9-4977-b551-e4daf9b9f74b"
-					(reference "#PWR344")
-					(unit 1)
-				)
-				(path "/5a60c4b1-b6cb-416e-8883-8291fa089b87/c2baf18d-2b19-4edb-98b3-535275ee271f/ed7a0d70-4012-4e50-88a7-aea647708582/4b0b4e20-0ae3-4a37-acd3-d6dca880b023"
-					(reference "#PWR256")
-					(unit 1)
-				)
-				(path "/5a60c4b1-b6cb-416e-8883-8291fa089b87/c2baf18d-2b19-4edb-98b3-535275ee271f/fb5bb440-61c9-4bd3-9ab6-a463ad90c8bb/413450a6-23f7-43dd-83b0-93f1b2a57e6d"
-					(reference "#PWR217")
-					(unit 1)
-				)
-			)
-			(project "analog_frontend_panel"
-				(path "/c241d083-1323-4b4a-a540-956d0afb7b72/19141585-7846-417a-91df-f61215fe3233/413450a6-23f7-43dd-83b0-93f1b2a57e6d"
-					(reference "#PWR17002")
-					(unit 1)
-				)
-				(path "/c241d083-1323-4b4a-a540-956d0afb7b72/1fbd3e63-3701-4f31-b722-16e65c25cea8/413450a6-23f7-43dd-83b0-93f1b2a57e6d"
-					(reference "#PWR18002")
-					(unit 1)
-				)
-				(path "/c241d083-1323-4b4a-a540-956d0afb7b72/3b63f70a-358c-4846-8cdc-f459df41a6c2/0ab125f9-c5b5-4162-87a8-3c0a237e613b"
-					(reference "#PWR25001")
-					(unit 1)
-				)
-				(path "/c241d083-1323-4b4a-a540-956d0afb7b72/77831b95-4af9-4be7-883d-350d130a19a2/4b0b4e20-0ae3-4a37-acd3-d6dca880b023"
-					(reference "#PWR30002")
-					(unit 1)
-				)
-				(path "/c241d083-1323-4b4a-a540-956d0afb7b72/b7e73f80-a01f-409c-a1ae-634c4b865833/4b0b4e20-0ae3-4a37-acd3-d6dca880b023"
-					(reference "#PWR28001")
-					(unit 1)
-				)
-				(path "/c241d083-1323-4b4a-a540-956d0afb7b72/be220027-a1e7-4f8a-b4af-8d208623fd51/dd604314-47f9-4977-b551-e4daf9b9f74b"
-					(reference "#PWR24002")
-					(unit 1)
-				)
-				(path "/c241d083-1323-4b4a-a540-956d0afb7b72/c0b9347d-9aa2-441c-987f-68119b1d92c1/0ab125f9-c5b5-4162-87a8-3c0a237e613b"
-					(reference "#PWR21002")
-					(unit 1)
-				)
-				(path "/c241d083-1323-4b4a-a540-956d0afb7b72/c99c1b0b-6659-4cec-a152-edd7ebc08576/4b0b4e20-0ae3-4a37-acd3-d6dca880b023"
-					(reference "#PWR16002")
-					(unit 1)
-				)
-				(path "/c241d083-1323-4b4a-a540-956d0afb7b72/ed2f7b43-1244-451f-9def-7c9639b384e1/dd604314-47f9-4977-b551-e4daf9b9f74b"
-					(reference "#PWR42003")
-					(unit 1)
-				)
-				(path "/c241d083-1323-4b4a-a540-956d0afb7b72/ed7a0d70-4012-4e50-88a7-aea647708582/4b0b4e20-0ae3-4a37-acd3-d6dca880b023"
-					(reference "#PWR31003")
-					(unit 1)
-				)
-				(path "/c241d083-1323-4b4a-a540-956d0afb7b72/fb5bb440-61c9-4bd3-9ab6-a463ad90c8bb/413450a6-23f7-43dd-83b0-93f1b2a57e6d"
-					(reference "#PWR15002")
 					(unit 1)
 				)
@@
 		(on_board yes)
 		(dnp no)
-		(property "Reference" "#PWR242"
+		(property "Reference" "#PWR301"
 			(at 124.46 77.47 0)
 			(effects
@@
 		(on_board yes)
 		(dnp no)
-		(property "Reference" "Q27002"
+		(property "Reference" "Q35002"
 			(at 92.964 91.44 90)
 			(effects
@@
 		(on_board yes)
 		(dnp no)
-		(property "Reference" "U27001"
+		(property "Reference" "U35001"
 			(at 107.442 78.994 0)
 			(effects
@@
 		(on_board yes)
 		(dnp no)
-		(property "Reference" "R27002"
+		(property "Reference" "R35002"
 			(at 93.98 77.343 90)
 			(effects
@@
 		(on_board yes)
 		(dnp no)
-		(property "Reference" "C27003"
+		(property "Reference" "C35003"
 			(at 119.38 81.788 90)
 			(effects
@@
 		(on_board yes)
 		(dnp no)
-		(property "Reference" "C27004"
+		(property "Reference" "C35004"
 			(at 118.872 97.536 90)
 			(effects
@@
 		(on_board yes)
 		(dnp no)
-		(property "Reference" "C27002"
+		(property "Reference" "C35002"
 			(at 111.252 65.532 90)
 			(effects
@@
 		(on_board yes)
 		(dnp no)
-		(property "Reference" "#PWR243"
+		(property "Reference" "#PWR304"
 			(at 113.03 81.28 0)
 			(effects
@@
 		(on_board yes)
 		(dnp no)
-		(property "Reference" "#PWR185"
+		(property "Reference" "#PWR205"
 			(at 101.6 99.06 0)
 			(effects

Commit message: schematic updates for ovp rail and dac pulldown
Parts:
- renumbered C35001 to C29001, C35002 to C29002, C35003 to C29003, C35004 to C29004, Q35001 to Q29001, Q35002 to Q29002, R43001 to R21001, R35002 to R29002, U35001 to U29001
Changed lines of the file:
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@@
 		(on_board yes)
 		(dnp no)
-		(property "Reference" "#PWR309"
+		(property "Reference" "#PWR257"
 			(at 113.03 88.9 0)
 			(effects
@@
 		(on_board yes)
 		(dnp no)
-		(property "Reference" "C35001"
+		(property "Reference" "C29001"
 			(at 106.68 96.012 90)
 			(effects
@@
 		(on_board yes)
 		(dnp no)
-		(property "Reference" "#PWR305"
+		(property "Reference" "#PWR255"
 			(at 92.964 110.49 0)
 			(effects
@@
 		(on_board yes)
 		(dnp no)
-		(property "Reference" "R43001"
+		(property "Reference" "R21001"
 			(at 82.55 77.343 90)
 			(effects
@@
 		(on_board yes)
 		(dnp no)
-		(property "Reference" "#PWR300"
+		(property "Reference" "#PWR252"
 			(at 124.46 92.71 0)
 			(effects
@@
 		(on_board yes)
 		(dnp no)
-		(property "Reference" "Q35001"
+		(property "Reference" "Q29001"
 			(at 80.772 100.584 90)
 			(effects
@@
 		(on_board yes)
 		(dnp no)
-		(property "Reference" "#PWR301"
+		(property "Reference" "#PWR253"
 			(at 124.46 77.47 0)
 			(effects
@@
 		(on_board yes)
 		(dnp no)
-		(property "Reference" "Q35002"
+		(property "Reference" "Q29002"
 			(at 92.964 91.44 90)
 			(effects
@@
 		(on_board yes)
 		(dnp no)
-		(property "Reference" "U35001"
+		(property "Reference" "U29001"
 			(at 107.442 78.994 0)
 			(effects
@@
 		(on_board yes)
 		(dnp no)
-		(property "Reference" "R35002"
+		(property "Reference" "R29002"
 			(at 93.98 77.343 90)
 			(effects
@@
 		(on_board yes)
 		(dnp no)
-		(property "Reference" "C35003"
+		(property "Reference" "C29003"
 			(at 119.38 81.788 90)
 			(effects
@@
 		(on_board yes)
 		(dnp no)
-		(property "Reference" "C35004"
+		(property "Reference" "C29004"
 			(at 118.872 97.536 90)
 			(effects
@@
 		(on_board yes)
 		(dnp no)
-		(property "Reference" "C35002"
+		(property "Reference" "C29002"
 			(at 111.252 65.532 90)
 			(effects
@@
 		(on_board yes)
 		(dnp no)
-		(property "Reference" "#PWR304"
+		(property "Reference" "#PWR254"
 			(at 113.03 81.28 0)
 			(effects
@@
 		(on_board yes)
 		(dnp no)
-		(property "Reference" "#PWR205"
+		(property "Reference" "#PWR190"
 			(at 101.6 99.06 0)
 			(effects

Commit message: set LCSC PNs for new connectors. wip to update layout for changes to ovp and dac
Parts:
- renumbered C29001 to C21001, C29002 to C21002, C29003 to C21003, C29004 to C21004, Q29001 to Q21001, Q29002 to Q21002, R29002 to R21002, R21001 to R24001, U29001 to U21001
Changed lines of the file:
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@@
 		(on_board yes)
 		(dnp no)
-		(property "Reference" "#PWR257"
+		(property "Reference" "#PWR220"
 			(at 113.03 88.9 0)
 			(effects
@@
 		(on_board yes)
 		(dnp no)
-		(property "Reference" "C29001"
+		(property "Reference" "C21001"
 			(at 106.68 96.012 90)
 			(effects
@@
 		(on_board yes)
 		(dnp no)
-		(property "Reference" "#PWR255"
+		(property "Reference" "#PWR216"
 			(at 92.964 110.49 0)
 			(effects
@@
 		(on_board yes)
 		(dnp no)
-		(property "Reference" "R21001"
+		(property "Reference" "R24001"
 			(at 82.55 77.343 90)
 			(effects
@@
 		(on_board yes)
 		(dnp no)
-		(property "Reference" "#PWR252"
+		(property "Reference" "#PWR208"
 			(at 124.46 92.71 0)
 			(effects
@@
 		(on_board yes)
 		(dnp no)
-		(property "Reference" "Q29001"
+		(property "Reference" "Q21001"
 			(at 80.772 100.584 90)
 			(effects
@@
 		(on_board yes)
 		(dnp no)
-		(property "Reference" "#PWR253"
+		(property "Reference" "#PWR209"
 			(at 124.46 77.47 0)
 			(effects
@@
 		(on_board yes)
 		(dnp no)
-		(property "Reference" "Q29002"
+		(property "Reference" "Q21002"
 			(at 92.964 91.44 90)
 			(effects
@@
 		(on_board yes)
 		(dnp no)
-		(property "Reference" "U29001"
+		(property "Reference" "U21001"
 			(at 107.442 78.994 0)
 			(effects
@@
 		(on_board yes)
 		(dnp no)
-		(property "Reference" "R29002"
+		(property "Reference" "R21002"
 			(at 93.98 77.343 90)
 			(effects
@@
 		(on_board yes)
 		(dnp no)
-		(property "Reference" "C29003"
+		(property "Reference" "C21003"
 			(at 119.38 81.788 90)
 			(effects
@@
 		(on_board yes)
 		(dnp no)
-		(property "Reference" "C29004"
+		(property "Reference" "C21004"
 			(at 118.872 97.536 90)
 			(effects
@@
 		(on_board yes)
 		(dnp no)
-		(property "Reference" "C29002"
+		(property "Reference" "C21002"
 			(at 111.252 65.532 90)
 			(effects
@@
 		(on_board yes)
 		(dnp no)
-		(property "Reference" "#PWR254"
+		(property "Reference" "#PWR212"
 			(at 113.03 81.28 0)
 			(effects
@@
 		(on_board yes)
 		(dnp no)
-		(property "Reference" "#PWR190"
+		(property "Reference" "#PWR169"
 			(at 101.6 99.06 0)
 			(effects

Commit message: update notes for clamp voltage
Parts:
- renumbered C21001 to C45001, C21002 to C45002, C21003 to C45003, C21004 to C45004, Q21001 to Q45001, Q21002 to Q45002, R24001 to R31001, R21002 to R45002, U21001 to U45001
Other:
- note added: "JFETs in diode arrangement are used for their extremely low leakage current, because leakage current here causes error in measured voltage. Expect about 0.6V forward voltage which gives a clamping range of [-0.6, 3.1] V in this case. TI application note AB-064 describes the approach in more detail. https://www.ti.com/lit/an/sboa058/sboa058.pdf"
- note removed: "JFETs in diode arrangement are used for their extremely low leakage current, because leakage current here causes error in measured voltage. Expect about 0.6V forward voltage which gives a clamping range of [-0.6, 3.9] V in this case. TI application note AB-064 describes the approach in more detail. https://www.ti.com/lit/an/sboa058/sboa058.pdf"
Changed lines of the file:
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@@
 		)
 	)
-	(text "JFETs in diode arrangement\nare used for their extremely\nlow leakage current, because\nleakage current here causes\nerror in measured voltage.\n\nExpect about 0.6V forward voltage\nwhich gives a clamping range of\n[-0.6, 3.9] V in this case.\n\nTI application note AB-064\ndescribes the approach in more\ndetail.\n\nhttps://www.ti.com/lit/an/sboa058/sboa058.pdf"
+	(text "JFETs in diode arrangement\nare used for their extremely\nlow leakage current, because\nleakage current here causes\nerror in measured voltage.\n\nExpect about 0.6V forward voltage\nwhich gives a clamping range of\n[-0.6, 3.1] V in this case.\n\nTI application note AB-064\ndescribes the approach in more\ndetail.\n\nhttps://www.ti.com/lit/an/sboa058/sboa058.pdf"
 		(exclude_from_sim no)
 		(at 73.152 125.984 0)
@@
 		(on_board yes)
 		(dnp no)
-		(property "Reference" "#PWR220"
+		(property "Reference" "#PWR351"
 			(at 113.03 88.9 0)
 			(effects
@@
 		(on_board yes)
 		(dnp no)
-		(property "Reference" "C21001"
+		(property "Reference" "C45001"
 			(at 106.68 96.012 90)
 			(effects
@@
 		(on_board yes)
 		(dnp no)
-		(property "Reference" "#PWR216"
+		(property "Reference" "#PWR349"
 			(at 92.964 110.49 0)
 			(effects
@@
 		(on_board yes)
 		(dnp no)
-		(property "Reference" "R24001"
+		(property "Reference" "R31001"
 			(at 82.55 77.343 90)
 			(effects
@@
 		(on_board yes)
 		(dnp no)
-		(property "Reference" "#PWR208"
+		(property "Reference" "#PWR346"
 			(at 124.46 92.71 0)
 			(effects
@@
 		(on_board yes)
 		(dnp no)
-		(property "Reference" "Q21001"
+		(property "Reference" "Q45001"
 			(at 80.772 100.584 90)
 			(effects
@@
 		(on_board yes)
 		(dnp no)
-		(property "Reference" "#PWR209"
+		(property "Reference" "#PWR347"
 			(at 124.46 77.47 0)
 			(effects
@@
 		(on_board yes)
 		(dnp no)
-		(property "Reference" "Q21002"
+		(property "Reference" "Q45002"
 			(at 92.964 91.44 90)
 			(effects
@@
 		(on_board yes)
 		(dnp no)
-		(property "Reference" "U21001"
+		(property "Reference" "U45001"
 			(at 107.442 78.994 0)
 			(effects
@@
 		(on_board yes)
 		(dnp no)
-		(property "Reference" "R21002"
+		(property "Reference" "R45002"
 			(at 93.98 77.343 90)
 			(effects
@@
 		(on_board yes)
 		(dnp no)
-		(property "Reference" "C21003"
+		(property "Reference" "C45003"
 			(at 119.38 81.788 90)
 			(effects
@@
 		(on_board yes)
 		(dnp no)
-		(property "Reference" "C21004"
+		(property "Reference" "C45004"
 			(at 118.872 97.536 90)
 			(effects
@@
 		(on_board yes)
 		(dnp no)
-		(property "Reference" "C21002"
+		(property "Reference" "C45002"
 			(at 111.252 65.532 90)
 			(effects
@@
 		(on_board yes)
 		(dnp no)
-		(property "Reference" "#PWR212"
+		(property "Reference" "#PWR348"
 			(at 113.03 81.28 0)
 			(effects
@@
 		(on_board yes)
 		(dnp no)
-		(property "Reference" "#PWR169"
+		(property "Reference" "#PWR250"
 			(at 101.6 99.06 0)
 			(effects
