File: hardware/boards/deimos_daq_rev7/analog/sk_3kHz.kicad_sch (KiCad schematic)
At the start: 9 parts, among them Q45001 MMBFJ113, Q45002 MMBFJ113, U45001 OPA196xDBV

Commit message: wip to export more gpio pins
Parts:
- renumbered C45001 to C27001, C45002 to C27002, C45003 to C27003, C45004 to C27004, Q45001 to Q27001, Q45002 to Q27002, R31001 to R27001, R45002 to R27002, U45001 to U27001
Changed lines of the file:
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@@
 		(on_board yes)
 		(dnp no)
-		(property "Reference" "#PWR351"
+		(property "Reference" "#PWR246"
 			(at 113.03 88.9 0)
 			(effects
@@
 		(on_board yes)
 		(dnp no)
-		(property "Reference" "C45001"
+		(property "Reference" "C27001"
 			(at 106.68 96.012 90)
 			(effects
@@
 		(on_board yes)
 		(dnp no)
-		(property "Reference" "#PWR349"
+		(property "Reference" "#PWR244"
 			(at 92.964 110.49 0)
 			(effects
@@
 		(on_board yes)
 		(dnp no)
-		(property "Reference" "R31001"
+		(property "Reference" "R27001"
 			(at 82.55 77.343 90)
 			(effects
@@
 		(on_board yes)
 		(dnp no)
-		(property "Reference" "#PWR346"
+		(property "Reference" "#PWR239"
 			(at 124.46 92.71 0)
 			(effects
@@
 		(on_board yes)
 		(dnp no)
-		(property "Reference" "Q45001"
+		(property "Reference" "Q27001"
 			(at 80.772 100.584 90)
 			(effects
@@
 		(on_board yes)
 		(dnp no)
-		(property "Reference" "#PWR347"
+		(property "Reference" "#PWR242"
 			(at 124.46 77.47 0)
 			(effects
@@
 		(on_board yes)
 		(dnp no)
-		(property "Reference" "Q45002"
+		(property "Reference" "Q27002"
 			(at 92.964 91.44 90)
 			(effects
@@
 		(on_board yes)
 		(dnp no)
-		(property "Reference" "U45001"
+		(property "Reference" "U27001"
 			(at 107.442 78.994 0)
 			(effects
@@
 		(on_board yes)
 		(dnp no)
-		(property "Reference" "R45002"
+		(property "Reference" "R27002"
 			(at 93.98 77.343 90)
 			(effects
@@
 		(on_board yes)
 		(dnp no)
-		(property "Reference" "C45003"
+		(property "Reference" "C27003"
 			(at 119.38 81.788 90)
 			(effects
@@
 		(on_board yes)
 		(dnp no)
-		(property "Reference" "C45004"
+		(property "Reference" "C27004"
 			(at 118.872 97.536 90)
 			(effects
@@
 		(on_board yes)
 		(dnp no)
-		(property "Reference" "C45002"
+		(property "Reference" "C27002"
 			(at 111.252 65.532 90)
 			(effects
@@
 		(on_board yes)
 		(dnp no)
-		(property "Reference" "#PWR348"
+		(property "Reference" "#PWR243"
 			(at 113.03 81.28 0)
 			(effects
@@
 		(on_board yes)
 		(dnp no)
-		(property "Reference" "#PWR250"
+		(property "Reference" "#PWR185"
 			(at 101.6 99.06 0)
 			(effects
