File: hardware/boards/deimos_daq_rev7/analog/sk_3kHz.kicad_sch (KiCad schematic)
At the start: 9 parts, among them Q27001 MMBFJ113, Q27002 MMBFJ113, U27001 OPA196xDBV

Commit message: Rev 7.0.3 hardware (#64)
## 2026-08-14 Hardware Rev 7.0.3

* [x] Flip orientation of IDC header
* [x] Resolve crosstalk between 35mV channels and thermocouple channels
    * Buffer shared 1.024V offset ref at each 35mV frontend
* [x] Improve light-pipe LED brightness
* [x] Improve 24V supply filtering
* Need better immunity to conducted EMI from the upstream power supply
    * Just added more capacitance for now
* [x] Exclude testpoints from BOM
Parts:
- renumbered C27001 to C31001, C27002 to C31002, C27003 to C31003, C27004 to C31004, Q27001 to Q31001, Q27002 to Q31002, R27001 to R31001, R27002 to R31002, U27001 to U31001
Changed lines of the file:
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@@
 		(on_board yes)
 		(dnp no)
-		(property "Reference" "#PWR246"
+		(property "Reference" "#PWR271"
 			(at 113.03 88.9 0)
 			(effects
@@
 		(on_board yes)
 		(dnp no)
-		(property "Reference" "C27001"
+		(property "Reference" "C31001"
 			(at 106.68 96.012 90)
 			(effects
@@
 		(on_board yes)
 		(dnp no)
-		(property "Reference" "#PWR244"
+		(property "Reference" "#PWR268"
 			(at 92.964 110.49 0)
 			(effects
@@
 		(on_board yes)
 		(dnp no)
-		(property "Reference" "R27001"
+		(property "Reference" "R31001"
 			(at 82.55 77.343 90)
 			(effects
@@
 		(on_board yes)
 		(dnp no)
-		(property "Reference" "#PWR239"
+		(property "Reference" "#PWR263"
 			(at 124.46 92.71 0)
 			(effects
@@
 		(on_board yes)
 		(dnp no)
-		(property "Reference" "Q27001"
+		(property "Reference" "Q31001"
 			(at 80.772 100.584 90)
 			(effects
@@
 		(on_board yes)
 		(dnp no)
-		(property "Reference" "#PWR242"
+		(property "Reference" "#PWR265"
 			(at 124.46 77.47 0)
 			(effects
@@
 		(on_board yes)
 		(dnp no)
-		(property "Reference" "Q27002"
+		(property "Reference" "Q31002"
 			(at 92.964 91.44 90)
 			(effects
@@
 		(on_board yes)
 		(dnp no)
-		(property "Reference" "U27001"
+		(property "Reference" "U31001"
 			(at 107.442 78.994 0)
 			(effects
@@
 		(on_board yes)
 		(dnp no)
-		(property "Reference" "R27002"
+		(property "Reference" "R31002"
 			(at 93.98 77.343 90)
 			(effects
@@
 		(on_board yes)
 		(dnp no)
-		(property "Reference" "C27003"
+		(property "Reference" "C31003"
 			(at 119.38 81.788 90)
 			(effects
@@
 		(on_board yes)
 		(dnp no)
-		(property "Reference" "C27004"
+		(property "Reference" "C31004"
 			(at 118.872 97.536 90)
 			(effects
@@
 		(on_board yes)
 		(dnp no)
-		(property "Reference" "C27002"
+		(property "Reference" "C31002"
 			(at 111.252 65.532 90)
 			(effects
@@
 		(on_board yes)
 		(dnp no)
-		(property "Reference" "#PWR243"
+		(property "Reference" "#PWR266"
 			(at 113.03 81.28 0)
 			(effects
@@
 		(on_board yes)
 		(dnp no)
-		(property "Reference" "#PWR185"
+		(property "Reference" "#PWR195"
 			(at 101.6 99.06 0)
 			(effects
