File: hardware/boards/deimos_daq_rev7/analog/ain_g25p7_.kicad_sch (KiCad schematic)
At the start: 6 parts, among them IC38001 INA826AIDR

Commit message: replace 660x channel with another 25.7x
Parts:
- renumbered C38001 to C36001, C38002 to C36002, C38003 to C36003, IC38001 to IC36001, R38001 to R36001, R38002 to R36002
