File: hardware/boards/deimos_daq_rev7/analog/analog_frontend_panel.kicad_pcb (KiCad board)
At the start: 4 copper layers, 371 parts, among them IC1 INA826AIDR, IC1002 BD42540FJ-CE2, IC12 INA826AIDR, IC13 TLV333IDBVR, IC14 TLV333IDBVR, IC14001 INA826AIDR, IC15 INA826AIDR, IC16 TLV333IDBVR, IC17 TLV333IDBVR, IC18 INA826AIDR, IC19 TLV333IDBVR, IC2 INA826AIDR, IC20 TLV333IDBVR, IC21 INA826AIDR, IC22 TLV333IDBVR, IC23 TLV333IDBVR, IC31001 INA826AIDR, IC32001 BD42540FJ-CE2, IC33001 BD42540FJ-CE2, IC34001 BD42540FJ-CE2, IC34002 INA826AIDR, IC35001 BD42540FJ-CE2, IC37001 INA826AIDR, J1001 WJ15EDGRM-3.81-12P, J1002 WJ15EDGRM-3.81-12P, J1003 WJ15EDGRM-3.81-12P, J1004 WJ15EDGRM-3.81-12P, J1005 WJ15EDGRM-3.81-12P, J1006 XG4C-2631, J1007 WJ15EDGRM-3.81-12P, J12 AM-K-PCB, J13 AM-K-PCB, Q15001 MMBFJ113, Q15002 MMBFJ113, Q16001 MMBFJ113, Q16002 MMBFJ113, Q17001 MMBFJ113, Q17002 MMBFJ113, Q18001 MMBFJ113, Q18002 MMBFJ113, Q20001 MMBFJ113, Q20002 MMBFJ113, Q21001 MMBFJ113, Q21002 MMBFJ113, Q24001 MMBFJ113, Q24002 MMBFJ113, Q25001 MMBFJ113, Q25002 MMBFJ113, Q28001 MMBFJ113, Q28002 MMBFJ113, Q28003 MMBFJ113, Q28004 MMBFJ113, Q30001 MMBFJ113, Q30002 MMBFJ113, Q31001 MMBFJ113, Q31002 MMBFJ113, Q42001 MMBFJ113, Q42002 MMBFJ113, Q5001 MMBFJ113, Q5002 MMBFJ113, Q8001 MMBFJ113, Q8002 MMBFJ113, Q9001 MMBFJ113, Q9002 MMBFJ113, U1 NTJD4001NT1G, U1001 ATL431BQDBZR, U15001 OPA196xDBV, U16001 OPA196xDBV, U17001 OPA196xDBV, U18001 OPA196xDBV, U2 NTJD4001NT1G, U20002 OPA196xDBV, U21001 OPA196xDBV, U24001 OPA196xDBV, U25001 OPA196xDBV, U28001 OPA196xDBV, U28002 OPA196xDBV, U3 NTJD4001NT1G, U30001 OPA196xDBV, U31001 OPA196xDBV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

Commit message: Deimos DAQ Rev 7.0.1 (#57)
## 2026-07-19 0.18.1

* Rev7 hardware
    * Finish pcb layout updates & re-generate fab files
    * Update enclosure graphics
* Rev7 firmware
    * Move `sample()` function with DSP pipeline into ITCM memory
    * Move `Net::poll` function with bulk of networking logic into ITCM
* This prevents them from being ejected from cache, or taking up space
in cache
* This should allow all remaining Operating-state code to remain in L1
cache (16kB)
* deimos
    * Update an example and reqwest dep
Routing:
- net +2V5: track 252.7 -> 215.7 mm
- net 2V5_OVP: track 291.8 -> 292.9 mm
Changed lines of the file:
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@@
 	)
 	(segment
-		(start 250.75 113.8)
-		(end 270.725 113.8)
-		(width 0.25)
-		(layer "F.Cu")
-		(net 3)
-	)
-	(segment
 		(start 270.9225 124.3705)
 		(end 270.9225 124.15887)
@@
 	)
 	(segment
-		(start 273.2625 108.1)
-		(end 273.9875 108.825)
-		(width 0.25)
-		(layer "F.Cu")
-		(net 3)
-	)
-	(segment
 		(start 189.385 120.39)
 		(end 186.5728 120.39)
@@
 	)
 	(segment
-		(start 249.55 115)
-		(end 250.75 113.8)
-		(width 0.25)
-		(layer "F.Cu")
-		(net 3)
-	)
-	(segment
 		(start 225.85 143.6521)
 		(end 226.6295 143.6521)
@@
 	)
 	(segment
-		(start 270.725 113.8)
-		(end 271.15 113.375)
-		(width 0.25)
-		(layer "F.Cu")
-		(net 3)
-	)
-	(segment
 		(start 224.6856 143.6521)
 		(end 225.7248 143.6521)
@@
 	)
 	(segment
-		(start 249.55 120.4)
-		(end 249.55 115)
-		(width 0.25)
-		(layer "F.Cu")
-		(net 3)
-	)
-	(segment
 		(start 263.9256 122.6464)
 		(end 263.9256 122.5956)
@@
 	)
 	(segment
-		(start 271.375 108.1)
-		(end 273.2625 108.1)
-		(width 0.25)
-		(layer "F.Cu")
-		(net 3)
-	)
-	(segment
 		(start 182.4704 148.3962)
 		(end 178.608 152.2586)
@@
 	)
 	(segment
-		(start 271.15 113.375)
-		(end 271.15 108.325)
-		(width 0.25)
-		(layer "F.Cu")
-		(net 3)
-	)
-	(segment
 		(start 190.585 121.117639)
 		(end 190.112639 121.117639)
@@
 	)
 	(segment
-		(start 250.325 121.175)
-		(end 249.55 120.4)
-		(width 0.25)
-		(layer "F.Cu")
-		(net 3)
-	)
-	(segment
 		(start 202.335 121.12617)
 		(end 190.585 121.117639)
@@
 	)
 	(segment
-		(start 271.15 108.325)
-		(end 271.375 108.1)
-		(width 0.25)
-		(layer "F.Cu")
-		(net 3)
-	)
-	(segment
 		(start 186.5728 120.39)
 		(end 182.4704 124.4924)
@@
 	)
 	(segment
+		(start 273.975 108.8375)
+		(end 273.9875 108.825)
+		(width 0.2)
+		(layer "F.Cu")
+		(net 213)
+	)
+	(segment
 		(start 274.1875 131.77)
 		(end 274.1875 130.85)
@@
 		(layer "F.Cu")
 		(net 213)
+	)
+	(segment
+		(start 273.975 109.875)
+		(end 273.975 108.8375)
+		(width 0.2)
+		(layer "F.Cu")
+		(net 213)

Commit message: remove cap from shunt reg
Parts:
- removed C1002: 0.1uF, Capacitor_SMD:C_0402_1005Metric
Routing:
- net GND: vias 205 -> 204
Changed lines of the file:
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@@
 		)
 	)
-	(footprint "Capacitor_SMD:C_0402_1005Metric"
-		(layer "F.Cu")
-		(at 274.05 112.025)
-		(descr "Capacitor SMD 0402 (1005 Metric), square (rectangular) end terminal, IPC_7351 nominal, (Body size source: IPC-SM-782 page 76, https://www.pcb-3d.com/wordpress/wp-content/uploads/ipc-sm-782a_amendment_1_and_2.pdf), generated with kicad-footprint-generator")
-		(tags "capacitor")
-		(property "Reference" "C1002"
-			(at 0 -1.16 0)
-			(layer "F.SilkS")
-			(hide yes)
-			(effects
-				(font
-					(size 1 1)
-					(thickness 0.15)
-				)
-			)
-		)
-		(property "Value" "0.1uF"
-			(at 0 1.16 0)
-			(layer "F.Fab")
-			(effects
-				(font
-					(size 1 1)
-					(thickness 0.15)
-				)
-			)
-		)
-		(property "Footprint" "Capacitor_SMD:C_0402_1005Metric"
-			(at 0 0 0)
-			(unlocked yes)
-			(layer "F.Fab")
-			(hide yes)
-			(effects
-				(font
-					(size 1.27 1.27)
-					(thickness 0.15)
-				)
-			)
-		)
-		(property "Datasheet" ""
-			(at 0 0 0)
-			(unlocked yes)
-			(layer "F.Fab")
-			(hide yes)
-			(effects
-				(font
-					(size 1.27 1.27)
-					(thickness 0.15)
-				)
-			)
-		)
-		(property "Description" ""
-			(at 0 0 0)
-			(unlocked yes)
-			(layer "F.Fab")
-			(hide yes)
-			(effects
-				(font
-					(size 1.27 1.27)
-					(thickness 0.15)
-				)
-			)
-		)
-		(property ki_fp_filters "C_*")
-		(sheetname "Root")
-		(sheetfile "analog_frontend_panel.kicad_sch")
-		(attr smd)
-		(fp_line
-			(start -0.107836 -0.36)
-			(end 0.107836 -0.36)
-			(stroke
-				(width 0.12)
-				(type solid)
-			)
-			(layer "F.SilkS")
-		)
-		(fp_line
-			(start -0.107836 0.36)
-			(end 0.107836 0.36)
-			(stroke
-				(width 0.12)
-				(type solid)
-			)
-			(layer "F.SilkS")
-		)
-		(fp_line
-			(start -0.91 -0.46)
-			(end 0.91 -0.46)
-			(stroke
-				(width 0.05)
-				(type solid)
-			)
-			(layer "F.CrtYd")
-		)
-		(fp_line
-			(start -0.91 0.46)
-			(end -0.91 -0.46)
-			(stroke
-				(width 0.05)
-				(type solid)
-			)
-			(layer "F.CrtYd")
-		)
-		(fp_line
-			(start 0.91 -0.46)
-			(end 0.91 0.46)
-			(stroke
-				(width 0.05)
-				(type solid)
-			)
-			(layer "F.CrtYd")
-		)
-		(fp_line
-			(start 0.91 0.46)
-			(end -0.91 0.46)
-			(stroke
-				(width 0.05)
-				(type solid)
-			)
-			(layer "F.CrtYd")
-		)
-		(fp_line
-			(start -0.5 -0.25)
-			(end 0.5 -0.25)
-			(stroke
-				(width 0.1)
-				(type solid)
-			)
-			(layer "F.Fab")
-		)
-		(fp_line
-			(start -0.5 0.25)
-			(end -0.5 -0.25)
-			(stroke
-				(width 0.1)
-				(type solid)
-			)
-			(layer "F.Fab")
-		)
-		(fp_line
-			(start 0.5 -0.25)
-			(end 0.5 0.25)
-			(stroke
-				(width 0.1)
-				(type solid)
-			)
-			(layer "F.Fab")
-		)
-		(fp_line
-			(start 0.5 0.25)
-			(end -0.5 0.25)
-			(stroke
-				(width 0.1)
-				(type solid)
-			)
-			(layer "F.Fab")
-		)
-		(fp_text user "${REFERENCE}"
-			(at 0 0 0)
-			(layer "F.Fab")
-			(effects
-				(font
-					(size 0.25 0.25)
-					(thickness 0.04)
-				)
-			)
-		)
-		(pad "1" smd roundrect
-			(at -0.48 0)
-			(size 0.56 0.62)
-			(layers "F.Cu" "F.Paste" "F.Mask")
-			(roundrect_rratio 0.25)
-			(net 1 "GND")
-			(pintype "passive")
-		)
-		(pad "2" smd roundrect
-			(at 0.48 0)
-			(size 0.56 0.62)
-			(layers "F.Cu" "F.Paste" "F.Mask")
-			(roundrect_rratio 0.25)
-			(net 213 "2V5_OVP")
-			(pintype "passive")
-		)
-		(model "${KICAD8_3DMODEL_DIR}/Capacitor_SMD.3dshapes/C_0402_1005Metric.wrl"
-			(offset
-				(xyz 0 0 0)
-			)
-			(scale
-				(xyz 1 1 1)
-			)
-			(rotate
-				(xyz 0 0 0)
-			)
-		)
-	)
 	(footprint "Resistor_SMD:R_0402_1005Metric"
 		(layer "F.Cu")
@@
 		(size 0.8)
 		(drill 0.4)
-		(layers "F.Cu" "B.Cu")
-		(free yes)
-		(net 1)
-	)
-	(via
-		(at 272.825 111.975)
-		(size 0.8)
-		(drill 0.4)
