File: hardware/boards/deimos_daq_rev7/analog/sk_100Hz.kicad_sch (KiCad schematic)
At the start: 9 parts, among them Q15001 MMBFJ113, Q15002 MMBFJ113, U15001 OPA196xDBV

Commit message: Improve power input filters (#67)
* Remove immediate input power caps to eliminate spark on connection
* Add 220nH filter inductors to each converter
* Add LCSC ref number to OPA196 schematic symbols
Parts:
- U15001: LCSC (none) -> C2060757
Changed lines of the file:
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@@
+			)
+		)
+		(property "LCSC" "C2060757"
+			(at 115.57 85.09 0)
+			(effects
+				(font
+					(size 1.27 1.27)
+				)
+				(hide yes)
 			)
 		)
