File: hardware/boards/deimos_daq_rev8/analog/analog_frontend_panel.kicad_sch (KiCad schematic)
At the start: 17 parts, among them IC3002 BD42540FJ-CE2, J3001 WJ15EDGRM-3.81-12P, J3002 WJ15EDGRM-3.81-12P, J3003 WJ15EDGRM-3.81-12P, J3004 WJ15EDGRM-3.81-12P, J3005 WJ15EDGRM-3.81-12P, J3006 WJ15EDGRM-3.81-12P, J3007 XG4C-2631, U3001 ATL431BQDBZR

Commit message: update gpio input buffer schematic to use 22k resistor and schottky to 3v3 instead of zener to ground
Connections:
- net GND: now also J3004.3, J3004.9; no longer J3004.10, J3004.4, J3004.8
- net pwm_in_buf/VIN: now also J3004.10; no longer J3004.9
- net pwm_in_buf2/VIN: now also J3004.5; no longer J3004.3
- net pwm_in_buf3/VIN: now also J3004.7; no longer J3004.5
- net pwm_in_buf4/VIN: now also J3004.8; no longer J3004.7
- net pwm_in_buf9/VIN: now reaches J3004.1
- net pwm_in_buf8/VIN: now reaches J3004.2
- new net pwm_in_buf5/VIN: J3004.4
- no-connect marks 6 -> 4
Other:
- added sheet pwm_in_buf5 (pwm_in_buf.kicad_sch)
- added sheet pwm_in_buf8 (pwm_in_buf.kicad_sch)
- added sheet pwm_in_buf9 (pwm_in_buf.kicad_sch)
- note added: "DAC & PWM Output"
- note added: "Encoder Input"
- note added: "GPIO"
- note removed: "DAC & PWM Output w/ OVP"
- note removed: "GPIO w/ OVP"
- note removed: "PWM Input w/ OVP"

Commit message: finish routing new encoder channels. spread nc channels on connectors and update enclosure graphics. only support 2-wire 4-20mA to protect ground.
Connections:
- net GND: no longer J3002.12, J3002.3, J3002.6, J3002.9
- net RTD Amp/R+: now also J3001.1; no longer J3001.4
- net RTD Amp/R-: now also J3001.2; no longer J3001.5
- net RTD Amp/W-: now also J3001.3; no longer J3001.6
- net RTD Amp1/R+: now also J3001.5; no longer J3001.7
- net RTD Amp1/R-: now also J3001.6; no longer J3001.8
- net RTD Amp1/W-: now also J3001.7; no longer J3001.9
- net RTD Amp2/R+: now also J3001.9; no longer J3001.10
- net RTD Amp2/R-: now also J3001.10; no longer J3001.11
- net RTD Amp2/W-: now also J3001.11; no longer J3001.12
- no-connect marks 4 -> 8
Other:
- note added: "4-20mA (2-Wire)"
- note removed: "4-20mA (2/3-Wire)"
